File: quantum_arcade_pcb/quantum_arcade_pcb.sch (KiCad schematic (older format))
At the start: 77 parts, among them J20 J20, Q17 2N3904, Y1 12.096MHz

Commit message: Finished the first 2 pages of schematics
Parts:
- added B_1: 137290, symbol quantum_arcade_pcb:137290
- added C74: 1uf, symbol Device:CP1_Small
- added CR6: 1N100, symbol Device:D
- added D_1, H/J_4: LS138, symbol quantum_arcade_pcb:LS138
- added E_1: LS244A, symbol quantum_arcade_pcb:LS244A
- added F/H_4: LS04, symbol Star_Wars_Vector_PCB:LS04
- added F_1: LS244B, symbol quantum_arcade_pcb:LS244B
- added F_5: LS32, symbol Star_Wars_Vector_PCB:LS32
- added J_4: LS02, symbol Star_Wars_Vector_PCB:LS02
- added K/L_1: 68000, symbol quantum_arcade_pcb:68000
- added K_4: LS08, symbol Star_Wars_Vector_PCB:LS08
- added L_4: LS74, symbol Star_Wars_Vector_PCB:LS74
- added L_6: LS14, symbol Star_Wars_Vector_PCB:LS14
- added M/N_12: TL082, symbol Amplifier_Operational:TL082
- added M_4: LS06, symbol Asteroids:LS06
- added N_1: LS245B, symbol quantum_arcade_pcb:LS245B
- added N_4: S32, symbol Star_Wars_Vector_PCB:LS32
- added P_1: LS245A, symbol quantum_arcade_pcb:LS245A
- added P_4: LS00, symbol Star_Wars_Vector_PCB:LS00
- added unit 1 of P_8
- added R173, R215: 10k, symbol Device:R_US
- added R174: 68k, symbol Device:R_US
- added R175: 15k, symbol Device:R_US
- added R176: 1k, symbol Device:R_US
- added R216: 4.6k, symbol Device:R_US
- added R217: 4.7k, symbol Device:R_US
- added R223: 220, symbol Device:R_US
- added R_4, UR_5: LS393, symbol Asteroids:LS393
- added R_6: LS161, symbol Star_Wars_Vector_PCB:LS161
- added TPRESET1, TPRESET2, TPWDDIS1: TP, symbol Star_Wars_Vector_PCB:TP
Connections:
- net +10V: now also C74.1, M/N_12.8 (V+), R173.2
- net +5V: now also B_1.20 (Vcc), CR6.1 (K), D_1.16 (VCC), E_1.20 (VCC), F/H_4.14 (VCC), F_1.20 (VCC), F_5.14 (VCC), H/J_4.16 (VCC), K/L_1.14 (VCC), K/L_1.49 (VCC), K_4.14 (VCC), L_4.14 (VCC), M/N_12.2 (-), N_1.20 (VCC), P_1.20 (VCC), P_4.14 (VCC), P_8.14 (VCC), R215.2, R216.1, R217.1, R_4.14 (VCC), R_6.16 (VCC), UR_5.14 (VCC)
- net 6M: now also K/L_1.15 (CLK)
- net 750KHZ: now also UR_5.1 (1CK)
- net GND: now also B_1.10 (GND), C74.2, D_1.8 (GND), E_1.1 (OEa), E_1.10 (GND), E_1.19 (OEb), F/H_4.7 (GND), F_1.1 (OEa), F_1.10 (GND), F_1.19 (OEb), F_5.7 (GND), H/J_4.5 (~G2B), H/J_4.8 (GND), K/L_1.16 (GND), K/L_1.53 (GND), K_4.7 (GND), L_4.12 (2D), L_4.7 (GND), M/N_12.4 (V-), N_1.10 (GND), N_1.19 (CE), P_1.10 (GND), P_1.19 (CE), P_4.7 (GND), P_8.7 (GND), R175.1, R223.1, R_4.7 (GND), R_6.3 (A), R_6.4 (B), R_6.6 (D), R_6.8 (GND), TPRESET1.1, TPRESET1.2, UR_5.7 (GND)
- net PR218: now also H/J_4.6 (G1), K/L_1.12 (~BBACK), K/L_1.13 (~BR), K/L_1.22 (~BERR), K/L_1.23 (~IPL2), K/L_1.24 (~IPL1)
- net PR219: now also L_4.1 (~1CLR), L_4.13 (~1CLR)
- net PR220: now also R220.2, R_6.10 (ET), R_6.5 (C), R_6.7 (EP)
- net ~POR: now also L_4.4 (~1PRE_), L_6.6, P_4.1, R_6.1 (C)
- new net: M/N_12.1, R174.1, R176.2, R223.2
- new net: M/N_12.3 (+), R173.1, R174.2, R175.2
- new net: CR6.2 (A), L_6.3, R176.1, TPRESET2.1, TPRESET2.2
- new net: L_6.4, L_6.5, R_4.2 (1CLR), UR_5.2 (1CLR)
- new net: R_4.1 (1CK), UR_5.6 (1QD)
- new net: P_4.3, R_4.12 (2CLR), UR_5.12 (2CLR)
- new net: R_4.13 (2CK), UR_5.8 (2QD)
- new net: R_4.6 (1QD), R_6.2 (CLK)
- new net: L_4.3 (1CLK), R_4.8 (2QD)
- new net: R_6.14 (QA), UR_5.13 (2CK)
- new net: L_4.11 (2CLK), P_8.1, R_6.15 (RCO)
- new net: P_8.2, R_6.9 (LD)
- new net: K_4.3, L_4.2 (1D)
- new net: L_4.5 (1Q), M_4.11, M_4.9
- new net: K_4.1, R215.1, TPWDDIS1.1, TPWDDIS1.2
- new net: B_1.13, K_4.5
- new net A1: E_1.13 (I1b), K/L_1.29 (A1)
- new net A10: F_1.17 (I3b), K/L_1.38 (A10)
- new net A11: E_1.15 (I2b), K/L_1.39 (A11)
- new net A12: F_1.6 (I2a), K/L_1.40 (A12)
- new net A13: E_1.6 (I2a), K/L_1.41 (A13)
- new net A14: D_1.1 (A), F_1.15 (I2b), K/L_1.42 (A14)
- new net A15: F_1.8 (I3a), K/L_1.43 (A15)
- new net A16: D_1.3 (C), H/J_4.2 (B), K/L_1.44 (A16)
- new net A17: H/J_4.3 (C), K/L_1.45 (A17)
- new net A18: B_1.7, K/L_1.46 (A18)
- new net A19: B_1.6, K/L_1.47 (A19)
- new net A2: E_1.11 (I0b), K/L_1.30 (A2)
- new net A20: B_1.5, K/L_1.48 (A20)
- new net A21: B_1.4, K/L_1.50 (A21)
- new net A22: B_1.3, D_1.5 (~G2B), K/L_1.51 (A22)
- new net A23: B_1.2, D_1.4 (~G2A), K/L_1.52 (A23)
- new net A3: F_1.13 (I1b), K/L_1.31 (A3)
- new net A4: F_1.11 (I0b), K/L_1.32 (A4)
- new net A5: E_1.2 (I0a), K/L_1.33 (A5)
- new net A6: F_1.2 (I0a), K/L_1.34 (A6)
- new net A7: E_1.17 (I3b), K/L_1.35 (A7)
- new net A8: E_1.4 (I1a), K/L_1.36 (A8)
- new net A9: F_1.4 (I1a), K/L_1.37 (A9)
- new net AB1: E_1.7 (O1b)
- new net AB10: F_1.3 (O3b)
- new net AB11: E_1.5 (O2b)
- new net AB12: F_1.14 (O2a)
- new net AB13: E_1.14 (O2a)
- new net AB14: F_1.5 (O2b)
- new net AB15: D_1.2 (B), F_1.12 (O3a), H/J_4.1 (A)
- new net AB2: E_1.9 (O0b)
- new net AB3: F_1.7 (O1b)
- new net AB4: F_1.9 (O0b)
- new net AB5: E_1.18 (O0a)
- new net AB6: F_1.18 (O0a)
- new net AB7: E_1.3 (O3b)
- new net AB8: E_1.16 (O1a)
- new net AB9: F_1.16 (O1a)
- new net AS: D_1.6 (G1), F/H_4.2
- new net CS: J_4.10
- new net D0: K/L_1.5 (D0), N_1.15 (B3)
- new net D1: K/L_1.4 (D1), N_1.14 (B4)
- new net D10: K/L_1.59 (D10), P_1.16 (B2)
- new net D11: K/L_1.58 (D11), P_1.15 (B3)
- new net D12: K/L_1.57 (D12), P_1.14 (B4)
- new net D13: K/L_1.56 (D13), P_1.13 (B5)
- new net D14: K/L_1.55 (D14), P_1.12 (B6)
- new net D15: K/L_1.54 (D15), P_1.11 (B7)
- new net D2: K/L_1.3 (D2), N_1.13 (B5)
- new net D3: K/L_1.2 (D3), N_1.12 (B6)
- new net D4: K/L_1.1 (D4), N_1.11 (B7)
- new net D5: K/L_1.64 (D5), N_1.18 (B0)
- new net D6: K/L_1.63 (D6), N_1.17 (B1)
- new net D7: K/L_1.62 (D7), N_1.16 (B2)
- new net D8: K/L_1.61 (D8), P_1.18 (B0)
- new net D9: K/L_1.60 (D9), P_1.17 (B1)
- new net DB0: N_1.5 (A3)
- new net DB1: N_1.6 (A4)
- new net DB10: P_1.4 (A2)
- new net DB11: P_1.5 (A3)
- new net DB12: P_1.6 (A4)
- new net DB13: P_1.7 (A5)
- new net DB14: P_1.8 (A6)
- new net DB15: P_1.9 (A7)
- new net DB2: N_1.7 (A5)
- new net DB3: N_1.8 (A6)
- new net DB4: N_1.9 (A7)
- new net DB5: N_1.2 (A0)
- new net DB6: N_1.3 (A1)
- new net DB7: N_1.4 (A2)
- new net DB8: P_1.2 (A0)
- new net DB9: P_1.3 (A1)
- new net E: K/L_1.20 (E)
- new net FC0: B_1.11, K/L_1.28 (FC0)
- new net FC1: B_1.9, K/L_1.27 (FC1)
- new net FC2: B_1.8, K/L_1.26 (FC2)
- new net R\~W: E_1.8 (I3a), K/L_1.9 (R/~W)
- new net R\~W~B: E_1.12 (O3a), F/H_4.11, F_5.2, N_1.1 (DIR), N_4.10, N_4.13, P_1.1 (DIR)
- new net ~AS: B_1.1, F/H_4.1, K/L_1.6 (~AS)
- new net ~COLORAM: F_5.1, H/J_4.13 (Y2)
- new net ~CONTROL: H/J_4.12 (Y3)
- new net ~DTACK: K/L_1.10 (~DTACK)
- new net ~DTACK2: K_4.6
- new net ~HALT: K/L_1.17 (~HALT), M_4.10, R216.2
- new net ~IRQ: K/L_1.25 (~IPL0), L_4.9 (2Q)
- new net ~I\O: B_1.18, H/J_4.4 (~G2A)
- new net ~I\OS: B_1.15, J_4.8
- new net ~LDS: K/L_1.8 (~LDS), N_4.9
- new net ~NVRAM: B_1.19
- new net ~RAM0: D_1.9 (Y6)
- new net ~RAM1: D_1.7 (Y7)
- new net ~RECALL: H/J_4.11 (Y4)
- new net ~RESET: K/L_1.18 (~RESET), M_4.8, R217.2
- new net ~RESET*: K_4.2, L_4.6 (~1Q)
- new net ~ROM0: D_1.15 (Y0)
- new net ~ROM1: D_1.14 (Y1)
- new net ~ROM2: D_1.13 (Y2)
- new net ~ROM3: D_1.12 (Y3)
- new net ~ROM4: D_1.11 (Y4)
- new net ~R~\WB: F/H_4.10
- new net ~SWITCHES: H/J_4.14 (Y1)
- new net ~TRACKBALL: H/J_4.15 (Y0)
- new net ~UDS: K/L_1.7 (~UDS), N_4.12
- new net ~VBUFEN: K_4.4
- new net ~VGGO: H/J_4.9 (Y6)
- new net ~VGRST: H/J_4.10 (Y5)
- new net ~VMA: J_4.9, K/L_1.19 (~VMA)
- new net ~VMEM: B_1.16
- new net ~VPA: B_1.12, K/L_1.21 (~VPA), L_4.10 (~1PRE_)
- new net ~WDCLR: H/J_4.7 (Y7), P_4.2
- new net ~WEU: N_4.11
- no-connect marks 1 -> 21
Other:
- note added: "ADDRESS BUS BUFFERS"
- note added: "ADDRESS DECODERS"
- note added: "BIDIRECTIONAL DATA\nBUS BUFFERS"
- note added: "CHECK THIS!!!"
- note added: "MICROPROCESSOR"
- note added: "POWER-ON RESET AND WATCHDOG"
- moved on the sheet: J20

Commit message: Worked on schematic
Parts:
- added U? (x4): 2KX8_RAM, symbol quantum_arcade_pcb:2KX8_RAM
Connections:
- net +5V: now also U?.24 (VCC), U?.24 (VCC), U?.24 (VCC), U?.24 (VCC)
- net AB1: now also U?.8 (A0), U?.8 (A0), U?.8 (A0), U?.8 (A0)
- net AB10: now also U?.22 (A9), U?.22 (A9), U?.22 (A9), U?.22 (A9)
- net AB11: now also U?.19 (A10), U?.19 (A10), U?.19 (A10), U?.19 (A10)
- net AB2: now also U?.7 (A1), U?.7 (A1), U?.7 (A1), U?.7 (A1)
- net AB3: now also U?.6 (A2), U?.6 (A2), U?.6 (A2), U?.6 (A2)
- net AB4: now also U?.5 (A3), U?.5 (A3), U?.5 (A3), U?.5 (A3)
- net AB5: now also U?.4 (A4), U?.4 (A4), U?.4 (A4), U?.4 (A4)
- net AB6: now also U?.3 (A5), U?.3 (A5), U?.3 (A5), U?.3 (A5)
- net AB7: now also U?.2 (A6), U?.2 (A6), U?.2 (A6), U?.2 (A6)
- net AB8: now also U?.1 (A7), U?.1 (A7), U?.1 (A7), U?.1 (A7)
- net AB9: now also U?.23 (A8), U?.23 (A8), U?.23 (A8), U?.23 (A8)
- net GND: now also U?.12 (GND), U?.12 (GND), U?.12 (GND), U?.12 (GND)
- net ~RAM0: now also U?.18 (~CE), U?.18 (~CE)
- net ~RAM1: now also U?.18 (~CE), U?.18 (~CE)
- net ~R~\WB: now also U?.20 (~OE), U?.20 (~OE), U?.20 (~OE), U?.20 (~OE)
- net ~WEU: now also U?.21 (~WE), U?.21 (~WE)
- new net MB0: U?.9 (D0), U?.9 (D0)
- new net MB1: U?.10 (D1), U?.10 (D1)
- new net MB10: U?.11 (D2), U?.11 (D2)
- new net MB11: U?.13 (D3), U?.13 (D3)
- new net MB12: U?.14 (D4), U?.14 (D4)
- new net MB13: U?.15 (D5), U?.15 (D5)
- new net MB14: U?.16 (D6), U?.16 (D6)
- new net MB15: U?.17 (D7), U?.17 (D7)
- new net MB2: U?.11 (D2), U?.11 (D2)
- new net MB3: U?.13 (D3), U?.13 (D3)
- new net MB4: U?.14 (D4), U?.14 (D4)
- new net MB5: U?.15 (D5), U?.15 (D5)
- new net MB6: U?.16 (D6), U?.16 (D6)
- new net MB7: U?.17 (D7), U?.17 (D7)
- new net MB8: U?.9 (D0), U?.9 (D0)
- new net MB9: U?.10 (D1), U?.10 (D1)
- new net ~WEL: U?.21 (~WE), U?.21 (~WE)
Other:
- note added: "PROGRAM RAM"
- moved on the sheet: B_1, D_1, F/H_4A, F/H_4E, F_5A, H/J_4, J20, J_4C, K_4B, N_4C, N_4D

Commit message: added schematic stuff
Parts:
- gave numbers to parts that had none: 4
Changed lines of the file:
@@
 ADDRESS DECODERS
 $Comp
-L quantum_arcade_pcb:2KX8_RAM U?
+L quantum_arcade_pcb:2KX8_RAM N_3
 U 1 1 6DD416E2
 P 39600 2075
-F 0 "U?" H 39600 2050 50  0000 C CNN
+F 0 "N_3" H 39600 2050 50  0000 C CNN
 F 1 "2KX8_RAM" H 39600 2125 50  0000 C CNN
 F 2 "" H 39600 2075 50  0001 C CNN
@@
 $EndComp
 $Comp
-L quantum_arcade_pcb:2KX8_RAM U?
+L quantum_arcade_pcb:2KX8_RAM M_3
 U 1 1 6DD43EC4
 P 41700 2075
-F 0 "U?" H 41700 2025 50  0000 C CNN
+F 0 "M_3" H 41700 2025 50  0000 C CNN
 F 1 "2KX8_RAM" H 41700 2100 50  0000 C CNN
 F 2 "" H 41700 2075 50  0001 C CNN
@@
 $EndComp
 $Comp
-L quantum_arcade_pcb:2KX8_RAM U?
+L quantum_arcade_pcb:2KX8_RAM N_2
 U 1 1 6DD45B39
 P 39700 4350
-F 0 "U?" H 39675 4325 50  0000 C CNN
+F 0 "N_2" H 39675 4325 50  0000 C CNN
 F 1 "2KX8_RAM" H 39700 4400 50  0000 C CNN
 F 2 "" H 39700 4350 50  0001 C CNN
@@
 $EndComp
 $Comp
-L quantum_arcade_pcb:2KX8_RAM U?
+L quantum_arcade_pcb:2KX8_RAM M_2
 U 1 1 6DD910C1
 P 41775 4350
-F 0 "U?" H 41775 4325 50  0000 C CNN
+F 0 "M_2" H 41775 4325 50  0000 C CNN
 F 1 "2KX8_RAM" H 41775 4400 50  0000 C CNN
 F 2 "" H 41775 4350 50  0001 C CNN
@@
 AB3
 $Comp
-L power:GND #PWR?
+L power:GND #PWR0193
 U 1 1 6DF28438
 P 39600 2775
-F 0 "#PWR?" H 39600 2525 50  0001 C CNN
+F 0 "#PWR0193" H 39600 2525 50  0001 C CNN
 F 1 "GND" H 39750 2700 50  0000 C CNN
 F 2 "" H 39600 2775 50  0001 C CNN
@@
 $EndComp
 $Comp
-L power:GND #PWR?
+L power:GND #PWR0194
 U 1 1 6DF2B542
 P 41700 2775
-F 0 "#PWR?" H 41700 2525 50  0001 C CNN
+F 0 "#PWR0194" H 41700 2525 50  0001 C CNN
 F 1 "GND" H 41850 2700 50  0000 C CNN
 F 2 "" H 41700 2775 50  0001 C CNN
@@
 $EndComp
 $Comp
-L power:GND #PWR?
+L power:GND #PWR0195
 U 1 1 6DF2B9C1
 P 39700 5050
-F 0 "#PWR?" H 39700 4800 50  0001 C CNN
+F 0 "#PWR0195" H 39700 4800 50  0001 C CNN
 F 1 "GND" H 39850 4975 50  0000 C CNN
 F 2 "" H 39700 5050 50  0001 C CNN
@@
 $EndComp
 $Comp
-L power:GND #PWR?
+L power:GND #PWR0196
 U 1 1 6DF2BDAC
 P 41775 5050
-F 0 "#PWR?" H 41775 4800 50  0001 C CNN
+F 0 "#PWR0196" H 41775 4800 50  0001 C CNN
 F 1 "GND" H 41925 4975 50  0000 C CNN
 F 2 "" H 41775 5050 50  0001 C CNN
@@
 $EndComp
 $Comp
-L power:+5V #PWR?
+L power:+5V #PWR0197
 U 1 1 6DF2F647
 P 39850 1425
-F 0 "#PWR?" H 39850 1275 50  0001 C CNN
+F 0 "#PWR0197" H 39850 1275 50  0001 C CNN
 F 1 "+5V" H 39950 1500 50  0000 C CNN
 F 2 "" H 39850 1425 50  0001 C CNN
@@
 $EndComp
 $Comp
-L power:+5V #PWR?
+L power:+5V #PWR0198
 U 1 1 6DF31483
 P 41950 1425
-F 0 "#PWR?" H 41950 1275 50  0001 C CNN
+F 0 "#PWR0198" H 41950 1275 50  0001 C CNN
 F 1 "+5V" H 42050 1500 50  0000 C CNN
 F 2 "" H 41950 1425 50  0001 C CNN
@@
 $EndComp
 $Comp
-L power:+5V #PWR?
+L power:+5V #PWR0199
 U 1 1 6DF32184
 P 39950 3700
-F 0 "#PWR?" H 39950 3550 50  0001 C CNN
+F 0 "#PWR0199" H 39950 3550 50  0001 C CNN
 F 1 "+5V" H 40050 3775 50  0000 C CNN
 F 2 "" H 39950 3700 50  0001 C CNN
@@
 $EndComp
 $Comp
-L power:+5V #PWR?
+L power:+5V #PWR0200
 U 1 1 6DF329E4
 P 42025 3700
-F 0 "#PWR?" H 42025 3550 50  0001 C CNN
+F 0 "#PWR0200" H 42025 3550 50  0001 C CNN
 F 1 "+5V" H 42125 3775 50  0000 C CNN
 F 2 "" H 42025 3700 50  0001 C CNN

Commit message: Completed 5 schematic pages out of 14
Parts:
- added B_12: MC1495LB, symbol quantum_arcade_pcb:MC1495LB
- added C19, C20, C26, C27, C28, C31, C33, C34, C35, C36: .1uF, Star_Wars_Vector_PCB:GenericComp, symbol Device:C
- added C21: .0018uF, Star_Wars_Vector_PCB:SmallCap, symbol Device:C
- added C25: .047uF, Star_Wars_Vector_PCB:CapYellow, symbol Device:C
- added C29: 39pf, Star_Wars_Vector_PCB:GenericComp, symbol Device:C
- added C30, C32: 100pf, Star_Wars_Vector_PCB:GenericComp, symbol Device:C
- added C_12: MC1495LA, symbol quantum_arcade_pcb:MC1495LA
- added D/E_12, D_10: 082, Star_Wars_Vector_PCB:DIP8, symbol Star_Wars_Vector_PCB:082
- added E_10: LF13201, Star_Wars_Vector_PCB:DIP16, symbol Star_Wars_Vector_PCB:LF13201
- added E_2, E_3, F_2, F_3, H/J_2, H/J_3, K_2, K_3, L_2, L_3: 8KX8_ROM, symbol quantum_arcade_pcb:8KX8_ROM
- added unit 3 of F/H_4
- added F/H_9: AM6012, Star_Wars_Vector_PCB:DIP20, symbol Star_Wars_Vector_PCB:AM6012
- added J_10: LS04, Star_Wars_Vector_PCB:DIP14, symbol Star_Wars_Vector_PCB:LS04
- added unit 1 of N_4
- added P_2, P_3: LS245C, symbol quantum_arcade_pcb:LS245C
- added unit 3 of P_4
- added R106, R58: 7.5K, Star_Wars_Vector_PCB:GenericComp, symbol Device:R
- added R54, R61: 680, Star_Wars_Vector_PCB:GenericComp, symbol Device:R
- added R55: 820, Star_Wars_Vector_PCB:GenericComp, symbol Device:R
- added R59, R62, R63: 470, Star_Wars_Vector_PCB:GenericComp, symbol Device:R
- added R60: 2.7k, Star_Wars_Vector_PCB:GenericComp, symbol Device:R
- added R64, R69, R70, R77: 2.2k, Star_Wars_Vector_PCB:GenericComp, symbol Device:R
- added R65, R66, R78, R79: 3.9k, Star_Wars_Vector_PCB:GenericComp, symbol Device:R
- added R67, R73: 10k, Star_Wars_Vector_PCB:GenericComp, symbol Device:R
- added R68, R72: 10k, Star_Wars_Vector_PCB:PotBlk, symbol Star_Wars_Vector_PCB-rescue:POT
- added R71: 5.6k, Star_Wars_Vector_PCB:GenericComp, symbol Device:R
- added R74: 2K, Star_Wars_Vector_PCB:PotBlk, symbol Star_Wars_Vector_PCB-rescue:POT
- added R75: 100k, Star_Wars_Vector_PCB:GenericComp, symbol Device:R
- added R76: 1.2k, Star_Wars_Vector_PCB:GenericComp, symbol Device:R
- added R80: 1k, Star_Wars_Vector_PCB:GenericComp, symbol Device:R
- added RV2: VDR, Star_Wars_Vector_PCB:GenericComp, symbol Device:Varistor
- added R_2: LS74, symbol Star_Wars_Vector_PCB:LS74
- added TPYOUT1: TP, Star_Wars_Vector_PCB:TEST_POINT, symbol Star_Wars_Vector_PCB:TP
Connections:
- net +15V: now also B_12.2, C26.2, C28.2, C33.2, C35.1, D/E_12.8 (VCC), D_10.8 (VCC), E_10.13, R69.2, R70.2, R80.1
- net +5V: now also C19.1, E_2.1 (VPP), E_2.27 (~PGM), E_2.28 (VCC), E_3.1 (VPP), E_3.27 (~PGM), E_3.28 (VCC), F/H_9.20 (VCC), F_2.1 (VPP), F_2.27 (~PGM), F_2.28 (VCC), F_3.1 (VPP), F_3.27 (~PGM), F_3.28 (VCC), H/J_2.1 (VPP), H/J_2.27 (~PGM), H/J_2.28 (VCC), H/J_3.1 (VPP), H/J_3.27 (~PGM), H/J_3.28 (VCC), J_10.14 (VCC), K_2.1 (VPP), K_2.27 (~PGM), K_2.28 (VCC), K_3.1 (VPP), K_3.27 (~PGM), K_3.28 (VCC), L_2.1 (VPP), L_2.27 (~PGM), L_2.28 (VCC), L_3.1 (VPP), L_3.27 (~PGM), L_3.28 (VCC), N_4.14 (VCC), P_2.20 (VCC), P_3.20 (VCC), R_2.14 (VCC)
- net +6V: now also B_12.1, C32.1, C_12.1
- net -15V: now also B_12.7, C20.2, C27.2, C31.2, C34.2, C36.1, C_12.7, D/E_12.4 (VSS), D_10.4 (VSS), E_10.4, F/H_9.17 (V-)
- net 6M: now also R_2.11 (2CLK), R_2.3 (1CLK)
- net A23: now also N_4.1
- net AB1: now also E_2.10 (A0), E_3.10 (A0), F_2.10 (A0), F_3.10 (A0), H/J_2.10 (A0), H/J_3.10 (A0), K_2.10 (A0), K_3.10 (A0), L_2.10 (A0), L_3.10 (A0)
- net AB10: now also E_2.24 (A9), E_3.24 (A9), F_2.24 (A9), F_3.24 (A9), H/J_2.24 (A9), H/J_3.24 (A9), K_2.24 (A9), K_3.24 (A9), L_2.24 (A9), L_3.24 (A9)
- net AB11: now also E_2.21 (A10), E_3.21 (A10), F_2.21 (A10), F_3.21 (A10), H/J_2.21 (A10), H/J_3.21 (A10), K_2.21 (A10), K_3.21 (A10), L_2.21 (A10), L_3.21 (A10)
- net AB12: now also E_2.23 (A11), E_3.23 (A11), F_2.23 (A11), F_3.23 (A11), H/J_2.23 (A11), H/J_3.23 (A11), K_2.23 (A11), K_3.23 (A11), L_2.23 (A11), L_3.23 (A11)
- net AB13: now also E_2.2 (A12), E_3.2 (A12), F_2.2 (A12), F_3.2 (A12), H/J_2.2 (A12), H/J_3.2 (A12), K_2.2 (A12), K_3.2 (A12), L_2.2 (A12), L_3.2 (A12)
- net AB2: now also E_2.9 (A1), E_3.9 (A1), F_2.9 (A1), F_3.9 (A1), H/J_2.9 (A1), H/J_3.9 (A1), K_2.9 (A1), K_3.9 (A1), L_2.9 (A1), L_3.9 (A1)
- net AB3: now also E_2.8 (A2), E_3.8 (A2), F_2.8 (A2), F_3.8 (A2), H/J_2.8 (A2), H/J_3.8 (A2), K_2.8 (A2), K_3.8 (A2), L_2.8 (A2), L_3.8 (A2)
- net AB4: now also E_2.7 (A3), E_3.7 (A3), F_2.7 (A3), F_3.7 (A3), H/J_2.7 (A3), H/J_3.7 (A3), K_2.7 (A3), K_3.7 (A3), L_2.7 (A3), L_3.7 (A3)
- net AB5: now also E_2.6 (A4), E_3.6 (A4), F_2.6 (A4), F_3.6 (A4), H/J_2.6 (A4), H/J_3.6 (A4), K_2.6 (A4), K_3.6 (A4), L_2.6 (A4), L_3.6 (A4)
- net AB6: now also E_2.5 (A5), E_3.5 (A5), F_2.5 (A5), F_3.5 (A5), H/J_2.5 (A5), H/J_3.5 (A5), K_2.5 (A5), K_3.5 (A5), L_2.5 (A5), L_3.5 (A5)
- net AB7: now also E_2.4 (A6), E_3.4 (A6), F_2.4 (A6), F_3.4 (A6), H/J_2.4 (A6), H/J_3.4 (A6), K_2.4 (A6), K_3.4 (A6), L_2.4 (A6), L_3.4 (A6)
- net AB8: now also E_2.3 (A7), E_3.3 (A7), F_2.3 (A7), F_3.3 (A7), H/J_2.3 (A7), H/J_3.3 (A7), K_2.3 (A7), K_3.3 (A7), L_2.3 (A7), L_3.3 (A7)
- net AB9: now also E_2.25 (A8), E_3.25 (A8), F_2.25 (A8), F_3.25 (A8), H/J_2.25 (A8), H/J_3.25 (A8), K_2.25 (A8), K_3.25 (A8), L_2.25 (A8), L_3.25 (A8)
- net AS: now also R_2.10 (~1PRE_)
- net DB0: now also P_3.16 (B2)
- net DB1: now also P_3.14 (B4)
- net DB10: now also P_2.12 (B6)
- net DB11: now also P_2.11 (B7)
- net DB12: now also P_2.13 (B5)
- net DB13: now also P_2.15 (B3)
- net DB14: now also P_2.17 (B1)
- net DB15: now also P_2.18 (B0)
- net DB2: now also P_3.12 (B6)
- net DB3: now also P_3.11 (B7)
- net DB4: now also P_3.13 (B5)
- net DB5: now also P_3.15 (B3)
- net DB6: now also P_3.17 (B1)
- net DB7: now also P_3.18 (B0)
- net DB8: now also P_2.16 (B2)
- net DB9: now also P_2.14 (B4)
- net GND: now also C19.2, C20.1, C21.1, C26.1, C27.1, C28.1, C31.1, C33.1, C34.1, C35.2, C36.2, D_10.3 (+), D_10.5 (+), E_10.5, E_2.14 (GND), E_3.14 (GND), F/H_9.1 (B1), F/H_9.12 (B12), F/H_9.13 (GND), F/H_9.19 (~IO), F_2.14 (GND), F_3.14 (GND), H/J_2.14 (GND), H/J_3.14 (GND), J_10.7 (GND), K_2.14 (GND), K_3.14 (GND), L_2.14 (GND), L_3.14 (GND), N_4.7 (GND), P_2.10 (GND), P_3.10 (GND), R55.1, R61.1, R63.1, R67.1, R68.1, R68.2, R72.1, R72.2, R78.1, R79.1, RV2.2, R_2.7 (GND)
- net MB0: now also E_3.11 (D0), F_3.11 (D0), H/J_3.11 (D0), K_3.11 (D0), L_3.11 (D0), P_3.4 (A2)
- net MB1: now also E_3.12 (D1), F_3.12 (D1), H/J_3.12 (D1), K_3.12 (D1), L_3.12 (D1), P_3.6 (A4)
- net MB10: now also E_2.13 (D2), F_2.13 (D2), H/J_2.13 (D2), K_2.13 (D2), L_2.13 (D2), P_2.8 (A6)
- net MB11: now also E_2.15 (D3), F_2.15 (D3), H/J_2.15 (D3), K_2.15 (D3), L_2.15 (D3), P_2.9 (A7)
- net MB12: now also E_2.16 (D4), F_2.16 (D4), H/J_2.16 (D4), K_2.16 (D4), L_2.16 (D4), P_2.7 (A5)
- net MB13: now also E_2.17 (D5), F_2.17 (D5), H/J_2.17 (D5), K_2.17 (D5), L_2.17 (D5), P_2.5 (A3)
- net MB14: now also E_2.18 (D6), F_2.18 (D6), H/J_2.18 (D6), K_2.18 (D6), L_2.18 (D6), P_2.3 (A1)
- net MB15: now also E_2.19 (D7), F_2.19 (D7), H/J_2.19 (D7), K_2.19 (D7), L_2.19 (D7), P_2.2 (A0)
- net MB2: now also E_3.13 (D2), F_3.13 (D2), H/J_3.13 (D2), K_3.13 (D2), L_3.13 (D2), P_3.8 (A6)
- net MB3: now also E_3.15 (D3), F_3.15 (D3), H/J_3.15 (D3), K_3.15 (D3), L_3.15 (D3), P_3.9 (A7)
- net MB4: now also E_3.16 (D4), F_3.16 (D4), H/J_3.16 (D4), K_3.16 (D4), L_3.16 (D4), P_3.7 (A5)
- net MB5: now also E_3.17 (D5), F_3.17 (D5), H/J_3.17 (D5), K_3.17 (D5), L_3.17 (D5), P_3.5 (A3)
- net MB6: now also E_3.18 (D6), F_3.18 (D6), H/J_3.18 (D6), K_3.18 (D6), L_3.18 (D6), P_3.3 (A1)
- net MB7: now also E_3.19 (D7), F_3.19 (D7), H/J_3.19 (D7), K_3.19 (D7), L_3.19 (D7), P_3.2 (A0)
- net MB8: now also E_2.11 (D0), F_2.11 (D0), H/J_2.11 (D0), K_2.11 (D0), L_2.11 (D0), P_2.4 (A2)
- net MB9: now also E_2.12 (D1), F_2.12 (D1), H/J_2.12 (D1), K_2.12 (D1), L_2.12 (D1), P_2.6 (A4)
- net PR218: now also R_2.1 (~1CLR), R_2.13 (~1CLR), R_2.4 (~1PRE_)
- net R\~W: now also P_2.1 (DIR), P_3.1 (DIR)
- net YOUT: now also D/E_12.1, D/E_12.2 (-), TPYOUT1.1, TPYOUT1.2
- net ~AS: now also N_4.2
- net ~DTACK: now also F/H_4.6, P_4.9
- net ~ROM0: now also E_2.20 (G), E_3.20 (G)
- net ~ROM1: now also F_2.20 (G), F_3.20 (G)
- net ~ROM2: now also H/J_2.20 (G), H/J_3.20 (G)
- net ~ROM3: now also K_2.20 (G), K_3.20 (G)
- net ~ROM4: now also L_2.20 (G), L_3.20 (G)
- net ~R~\WB: now also E_2.22 (E), E_3.22 (E), F_2.22 (E), F_3.22 (E), H/J_2.22 (E), H/J_3.22 (E), K_2.22 (E), K_3.22 (E), L_2.22 (E), L_3.22 (E)
- new net: N_4.3, R_2.2 (1D)
- new net: F/H_4.5, P_4.8
- new net: C21.2, R54.2
- new net: F/H_9.15 (VR-), R55.2
- new net: C25.1, D_10.7, E_10.11, E_10.3, R58.2
- new net: D_10.1, E_10.14, R106.1
- new net: D_10.2 (-), R106.2, R58.1
- new net: E_10.15, E_10.2, R59.2, R62.2
- new net: E_10.1, J_10.2
- new net: C_12.2, D/E_12.5 (+), R69.1, R71.2
- new net: C29.2, C30.2, C_12.14, D/E_12.6 (-), R70.1, R73.2
- new net: C29.1, C30.1, D/E_12.7, R73.1, R74.1, R74.2
- new net: D/E_12.3 (+), R74.3, RV2.1
- new net: C_12.10, R65.2
- new net: C_12.11, R65.1
- new net: C_12.12, C_12.8, R63.2
- new net: C_12.13, R67.2
- new net: C_12.3, R66.2
- new net: C_12.4, R60.2, R61.2
- new net: C_12.5, R64.2
- new net: C_12.6, R64.1
- new net: C_12.9, R59.1
- new net: B_12.10, R77.2
- new net: B_12.11, R77.1
- new net: B_12.12, B_12.8, R78.2
- new net: B_12.13, B_12.3, R79.2
- new net: B_12.4, B_12.9, R62.1
- new net: B_12.5, R75.2, R76.2
- new net: B_12.6, C32.2, R75.1, R76.1
- new net: R66.1, R68.3
- new net: R71.1, R72.3
- new net DVY10: F/H_9.3 (B3)
- new net DVY2: F/H_9.11 (B11)
- new net DVY3: F/H_9.10 (B10)
- new net DVY4: F/H_9.9 (B9)
- new net DVY5: F/H_9.8 (B8)
- new net DVY6: F/H_9.7 (B7)
- new net DVY7: F/H_9.6 (B6)
- new net DVY8: F/H_9.5 (B5)
- new net DVY9: F/H_9.4 (B4)
- new net INVERTY: E_10.16, J_10.1
- new net XCOR: R60.1
- new net YBIP: C25.2, D_10.6 (-), E_10.10, F/H_9.18 (IO)
- new net YCOR: B_12.14, R80.2
- new net YREF: F/H_9.14 (VR+), R54.1
- new net ~CENTER: E_10.9
- new net ~DVY11: F/H_9.2 (B2)
- new net ~MDTACL: P_2.19 (CE), P_3.19 (CE)
- new net ~MTDACK: P_4.10, R_2.12 (2D), R_2.5 (1Q)
- no-connect marks 21 -> 28
Other:
- note added: "DATA TRANSFER ACK GENERATOR"
- note added: "NOT LOADED"
- note added: "PROGRAM ROM"
- note added: "Y-Axis Output"
