File: quantum_arcade_pcb/quantum_arcade_pcb.sch (KiCad schematic (older format))
At the start: 178 parts, among them J20 J20, Q17 2N3904, Y1 12.096MHz

Commit message: Completed 6 schematic pages out of 14
Parts:
- added A_10, D/E_11: 082, Star_Wars_Vector_PCB:DIP8, symbol Star_Wars_Vector_PCB:082
- added B_10: LF13201, Star_Wars_Vector_PCB:DIP16, symbol Star_Wars_Vector_PCB:LF13201
- added B_11: MC1495LB, symbol quantum_arcade_pcb:MC1495LB
- added B_9: AM6012, Star_Wars_Vector_PCB:DIP20, symbol Star_Wars_Vector_PCB:AM6012
- added C10, C11, C14, C15, C16, C17, C18, C2, C3, C39, C40, C9: .1uF, Star_Wars_Vector_PCB:GenericComp, symbol Device:C
- added C12: 39pf, Star_Wars_Vector_PCB:GenericComp, symbol Device:C
- added C13: 100pf, Star_Wars_Vector_PCB:GenericComp, symbol Device:C
- added C37: 150pF, Star_Wars_Vector_PCB:CapBrown, symbol Device:C
- added C38: 39pF, Star_Wars_Vector_PCB:CapBrown, symbol Device:C
- added C4: .01uF, Star_Wars_Vector_PCB:SmallCap, symbol Device:C
- added C41: .01uF, Star_Wars_Vector_PCB:GenericComp, symbol Device:C
- added C42: 10pF, Star_Wars_Vector_PCB:CapBrown, symbol Device:C
- added C64, C65, C67, C68, C69, C70: .1uf, symbol Device:C
- added C8: .047uF, Star_Wars_Vector_PCB:CapYellow, symbol Device:C
- added CR1: 1N914, Star_Wars_Vector_PCB:GenericComp, symbol Device:D
- added C_11: MC1495LA, symbol quantum_arcade_pcb:MC1495LA
- added D_8: LS273, symbol quantum_arcade_pcb:LS273
- added D_9: DAC_8, Star_Wars_Vector_PCB:DIP16, symbol Star_Wars_Vector_PCB:DAC_8
- added unit 6 of J_10
- added M_9, N_9: LS244C, symbol quantum_arcade_pcb:LS244C
- added N_8, P_9: LS191A, symbol Star_Wars_Vector_PCB:LS191A
- added Q7: 2N3904, Star_Wars_Vector_PCB:GenericTrans, symbol Star_Wars_Vector_PCB-rescue:2N3904
- added Q8: 2N3906, Star_Wars_Vector_PCB:GenericTrans, symbol Star_Wars_Vector_PCB-rescue:2N3906
- added R149, R151, R152, R160, R161, R162: 470, symbol Device:R_US
- added R153, R155, R156, R157, R158, R159: 1k, symbol Device:R_US
- added R180, R181, R182, R183, R184, R185, R186, R187: 100K, Star_Wars_Vector_PCB:GenericComp, symbol Device:R
- added R26, R27: 820, Star_Wars_Vector_PCB:GenericComp, symbol Device:R
- added R30, R31, R85, R86, R89, R93, R95, R96: 7.5K, Star_Wars_Vector_PCB:GenericComp, symbol Device:R
- added R32, R33, R38, R51: 470, Star_Wars_Vector_PCB:GenericComp, symbol Device:R
- added R34: 2.7k, Star_Wars_Vector_PCB:GenericComp, symbol Device:R
- added R35: 680, Star_Wars_Vector_PCB:GenericComp, symbol Device:R
- added R36, R44, R45, R50: 2.2k, Star_Wars_Vector_PCB:GenericComp, symbol Device:R
- added R37, R39, R52: 3.9k, Star_Wars_Vector_PCB:GenericComp, symbol Device:R
- added R40, R46: 10k, Star_Wars_Vector_PCB:GenericComp, symbol Device:R
- added R41: 5.6k, Star_Wars_Vector_PCB:GenericComp, symbol Device:R
- added R42, R43: 10k, Star_Wars_Vector_PCB:PotBlk, symbol Star_Wars_Vector_PCB-rescue:POT
- added R47: 2K, Star_Wars_Vector_PCB:PotBlk, symbol Star_Wars_Vector_PCB-rescue:POT
- added R48: 100k, Star_Wars_Vector_PCB:GenericComp, symbol Device:R
- added R49: 1.5k, Star_Wars_Vector_PCB:GenericComp, symbol Device:R
- added R53: 1k, Star_Wars_Vector_PCB:GenericComp, symbol Device:R
- added R81: 15K, Star_Wars_Vector_PCB:GenericComp, symbol Device:R
- added R82: 1K, Star_Wars_Vector_PCB:GenericComp, symbol Device:R
- added R83: 10K, Star_Wars_Vector_PCB:GenericComp, symbol Device:R
- added R84: 560, Star_Wars_Vector_PCB:GenericComp, symbol Device:R
- added R87, R91: 7.5k, Star_Wars_Vector_PCB:GenericComp, symbol Device:R
- added R88, R92: 200, Star_Wars_Vector_PCB:PotBlk, symbol Star_Wars_Vector_PCB-rescue:POT
- added R90, R94: 100, Star_Wars_Vector_PCB:GenericComp, symbol Device:R
- added R97: 3.9K, Star_Wars_Vector_PCB:GenericComp, symbol Device:R
- added RV1: VDR, Star_Wars_Vector_PCB:GenericComp, symbol Device:Varistor
- added TPXOUT1: TP, Star_Wars_Vector_PCB:TEST_POINT, symbol Star_Wars_Vector_PCB:TP
- renumbered C36 to C35, C35 to C36
Connections:
- net +15V: now also A_10.8 (VCC), B_10.13, B_11.2, C11.2, C15.2, C18.1, C9.2, D/E_11.8 (VCC), Q8.1 (E), R44.2, R45.2, R53.1, R82.2, R95.1, R96.1
- net +5V: now also B_9.20 (VCC), C2.1, C39.1, D_8.20 (VCC), D_9.13 (V+), M_9.20 (VCC), N_9.20 (VCC), R149.2, R151.2, R152.2, R160.2, R161.2, R162.2
- net +6V: now also B_11.1, C_11.1
- net -15V: now also A_10.4 (VSS), B_10.4, B_11.7, B_9.17 (V-), C10.2, C14.2, C16.2, C17.1, C3.2, C40.1, C41.1, C_11.7, D/E_11.4 (VSS), D_9.3 (V-)
- net COINAUX: now also R159.2, R162.1
- net COINL: now also R151.1, R155.2
- net COINR: now also R152.1, R156.2
- net DB0: now also M_9.12 (O3a), N_9.12 (O3a)
- net DB1: now also M_9.14 (O2a), N_9.14 (O2a)
- net DB2: now also M_9.16 (O1a), N_9.16 (O1a)
- net DB3: now also M_9.18 (O0a), N_9.18 (O0a)
- net DB4: now also M_9.5 (O2b), N_9.5 (O2b)
- net DB5: now also M_9.3 (O3b), N_9.3 (O3b)
- net DB6: now also M_9.7 (O1b), N_9.7 (O1b)
- net DB7: now also M_9.9 (O0b), N_9.9 (O0b)
- net DVY2: now also D_8.18 (D7)
- net DVY3: now also D_8.17 (D6)
- net DVY4: now also D_8.8 (D3)
- net DVY5: now also D_8.7 (D2)
- net DVY6: now also D_8.4 (D1)
- net DVY7: now also D_8.3 (D0)
- net GND: now also A_10.3 (+), A_10.5 (+), B_10.5, B_9.1 (B1), B_9.12 (B12), B_9.13 (GND), B_9.19 (~IO), C10.1, C11.1, C14.1, C15.1, C16.1, C17.2, C18.2, C2.2, C3.1, C39.2, C4.1, C40.2, C42.1, C64.2, C65.2, C67.2, C68.2, C69.2, C70.2, C9.1, CR1.2 (A), D_8.10 (GND), D_9.2 (~IO), M_9.10 (GND), M_9.13 (I1b), N_9.10 (GND), Q7.1 (E), R180.2, R181.2, R182.2, R183.2, R184.1, R185.1, R186.1, R187.1, R27.1, R35.1, R38.1, R40.1, R42.1, R42.2, R43.1, R43.2, R51.1, R52.1, R84.1, R97.1, RV1.2
- net SELFTEST: now also R149.1, R153.2
- net START1: now also R158.2, R161.1
- net START2: now also R157.2, R160.1
- net XCOR: now also B_11.14, R53.2
- net XOUT: now also D/E_11.1, D/E_11.2 (-), TPXOUT1.1, TPXOUT1.2
- net YBIP: now also R88.1, R88.2
- net YCOR: now also R34.1
- net YREF: now also R90.1
- net ~CENTER: now also B_10.9
- net ~SWITCHES: now also M_9.1 (OEa), M_9.19 (OEb)
- net ~TRACKBALL: now also N_9.1 (OEa), N_9.19 (OEb)
- new net: C4.2, R26.2
- new net: B_9.15 (VR-), R27.2
- new net: A_10.7, B_10.11, B_10.3, C8.1, R30.2
- new net: A_10.1, B_10.14, R31.1
- new net: A_10.2 (-), R30.1, R31.2
- new net: B_10.15, B_10.2, R32.2, R33.2
- new net: B_10.1, J_10.12
- new net: C_11.2, D/E_11.5 (+), R41.2, R44.1
- new net: C12.2, C13.2, C_11.14, D/E_11.6 (-), R45.1, R46.2
- new net: C12.1, C13.1, D/E_11.7, R46.1, R47.1, R47.2
- new net: D/E_11.3 (+), R47.3, RV1.1
- new net: C_11.10, R37.2
- new net: C_11.11, R37.1
- new net: C_11.12, C_11.8, R38.2
- new net: C_11.13, R40.2
- new net: C_11.3, R39.2
- new net: C_11.4, R34.2, R35.2
- new net: C_11.5, R36.2
- new net: C_11.6, R36.1
- new net: C_11.9, R32.1
- new net: B_11.10, R50.2
- new net: B_11.11, R50.1
- new net: B_11.12, B_11.8, R51.2
- new net: B_11.13, B_11.3, R52.2
- new net: B_11.4, B_11.9, R33.1
- new net: B_11.5, R48.2, R49.2
- new net: B_11.6, R48.1, R49.1
- new net: R39.1, R42.3
- new net: R41.1, R43.3
- new net: D_8.2 (Q0), D_9.5 (B1), R180.1
- new net: D_8.5 (Q1), D_9.6 (B2), R181.1
- new net: D_8.6 (Q2), D_9.7 (B3), R182.1
- new net: D_8.9 (Q3), D_9.8 (B4), R183.1
- new net: D_8.16 (Q6), D_9.9 (B5), R184.2
- new net: D_8.19 (Q7), D_9.10 (B6), R185.2
- new net: D_8.12 (Q4), D_9.11 (B7), R186.2
- new net: D_8.15 (Q5), D_9.12 (B8), R187.2
- new net: C41.2, D_9.16 (C)
- new net: D_9.15 (VR-), R97.2
- new net: D_9.14 (VR+), R95.2, R96.2
- new net: C37.1, Q7.2 (B), R81.1
- new net: C38.2, Q7.3 (C), R82.1, R83.2
- new net: C38.1, Q8.2 (B), R83.1
- new net: Q8.3 (C), R84.2, R85.2, R86.2
- new net: C42.2, CR1.1 (K), D_9.4 (IO), R85.1, R86.1, R87.2, R89.2, R91.2, R93.2
- new net: R87.1, R88.3
- new net: R89.1, R90.2
- new net: R91.1, R92.3
- new net: R93.1, R94.2
- new net: C67.1, M_9.11 (I0b), R153.1
- new net: C64.1, M_9.15 (I2b), R156.1
- new net: C65.1, M_9.17 (I3b), R155.1
- new net: C68.1, M_9.2 (I0a), R157.1
- new net: C69.1, M_9.4 (I1a), R158.1
- new net: C70.1, M_9.8 (I3a), R159.1
- new net DISRST: D_8.1 (C)
- new net DVX10: B_9.3 (B3)
- new net DVX2: B_9.11 (B11)
- new net DVX3: B_9.10 (B10)
- new net DVX4: B_9.9 (B9)
- new net DVX5: B_9.8 (B8)
- new net DVX6: B_9.7 (B7)
- new net DVX7: B_9.6 (B6)
- new net DVX8: B_9.5 (B5)
- new net DVX9: B_9.4 (B4)
- new net DVY0: D_8.14 (D5)
- new net DVY1: D_8.13 (D4)
- new net INVERTX: B_10.16, J_10.13
- new net SCALELO: D_8.11 (CK)
- new net VCTR: C37.2, R81.2
- new net XBIP: A_10.6 (-), B_10.10, B_9.18 (IO), C8.2, R92.1, R92.2
- new net XREF: B_9.14 (VR+), R26.1, R94.1
- new net ~DVX11: B_9.2 (B2)
- new net ~VCTR: D_9.1 (TH)
- new net ~VHALT: M_9.6 (I2a)
- no-connect marks 28 -> 32
Other:
- note added: "COIN DOOR AND CONTROL PANEL INPUT"
- note added: "DAC Reference And Bipolar Current Sources"
- note added: "X-Axis Output"
- moved on the sheet: F/H_4C, N_4A, P_4C, R_2A, R_2B

Commit message: Completed 8 pages of schematics
Parts:
- added B_2/3, D_2/3: POKEY, symbol quantum_arcade_pcb:POKEY
- added C51, C61: 1000pf 100V, symbol Device:C
- added C52, C53, C54, C55, C56, C57, C58, C59, C60, C62: 1uf 50V, symbol Device:C
- added C71, C72, C73: .1uf, symbol Device:C
- added C83, C84, C85, C86, C87, C88, C89, C90: .01uf 25V, symbol Device:C
- added unit 2 of F/H_4
- added unit 4 of F_5
- added unit 6 of M_4
- added unit 1 of M_4
- added N_10, P_11: 4584B, symbol Star_Wars_Vector_PCB:LS14
- added unit 2 of N_4
- added N_5: LS273B, symbol quantum_arcade_pcb:LS273B
- added P_10: LS157B, symbol Star_Wars_Vector_PCB:LS157B
- added unit 4 of P_4
- added unit 2 of P_4
- added Q15, Q16: 2N6044, symbol Device:Q_NPN_BCE
- added R110, R111, R112, R113, R114, R115, R116, R117: 3.3k, symbol Device:R_US
- added R118, R120, R121, R122, R123, R124, R125, R126, R127, R128, R163: 10k, symbol Device:R_US
- added R119, R129, R166, R167, R168, R169, R170, R171, R172: 1k, symbol Device:R_US
- added R164, R165: 220, symbol Device:R_US
- added R_10: LS74, symbol Star_Wars_Vector_PCB:LS74
- added R_3: X2212, symbol quantum_arcade_pcb:X2212
- added SW1, SW2: SW_DIP_x08, symbol Switch:SW_DIP_x08
- M_4: value LS06 -> 06
Connections:
- net +5V: now also N_8.16 (VCC), P_9.16 (VCC), B_2/3.17 (VCC), D_2/3.17 (VCC), M_4.14 (VCC), N_10.14 (VCC), N_5.20 (VCC), P_10.16 (VCC), P_11.14 (VCC), R163.1, R166.1, R168.1, R170.2, R171.2, R172.2, R_10.14 (VCC), R_3.18 (VCC)
- net 1HORIZCLK: now also C55.2, C85.2, R112.2
- net 1HORIZDIR: now also C53.2, C83.2, R110.2
- net 1VERTCLK: now also C59.2, C89.2, R116.2
- net 1VERTDIR: now also C57.2, C87.2, R114.2
- net 2HORIZCLK: now also C56.2, C86.2, R113.2
- net 2HORIZDIR: now also C54.2, C84.2, R111.2
- net 2VERTCLK: now also C60.2, C90.2, R117.2
- net 2VERTDIR: now also C58.2, C88.2, R115.2
- net AB1: now also R_3.6 (A0)
- net AB2: now also R_3.5 (A1)
- net AB3: now also R_3.4 (A2)
- net AB4: now also R_3.3 (A3)
- net AB5: now also R_3.2 (A4)
- net AB6: now also R_3.1 (A5)
- net AB7: now also R_3.17 (A6)
- net AB8: now also R_3.16 (A7)
- net COINCONTL: now also C72.1, Q15.2 (C)
- net COINCONTR: now also C73.1, Q16.2 (C)
- net DB0: now also N_5.8 (D3), R_3.12 (IO1)
- net DB1: now also N_5.3 (D0), R_3.13 (IO2)
- net DB2: now also N_5.7 (D2), R_3.14 (IO3)
- net DB3: now also N_5.4 (D1), R_3.15 (IO4)
- net DB4: now also N_5.14 (D5)
- net DB5: now also N_5.13 (D4)
- net DB6: now also N_5.18 (D7)
- net DB7: now also N_5.17 (D6)
- net GND: now also N_8.1 (B), N_8.10 (C), N_8.15 (A), N_8.4 (G), N_8.8 (GND), N_8.9 (D), P_9.1 (B), P_9.10 (C), P_9.15 (A), P_9.4 (G), P_9.8 (GND), P_9.9 (D), B_2/3.1 (GND), C51.2, C52.2, C61.2, C62.2, C71.2, C72.2, C73.2, C83.1, C84.1, C85.1, C86.1, C87.1, C88.1, C89.1, C90.1, D_2/3.1 (GND), M_4.7 (GND), N_10.7 (GND), N_5.10 (GND), P_10.15 (E), P_10.8 (GND), P_11.7 (GND), Q15.3 (E), Q16.3 (E), R110.1, R111.1, R112.1, R113.1, R114.1, R115.1, R116.1, R117.1, R_10.7 (GND), R_3.8 (VSS), SW1.10, SW1.11, SW1.12, SW1.13, SW1.14, SW1.15, SW1.16, SW1.9, SW2.10, SW2.11, SW2.12, SW2.13, SW2.14, SW2.15, SW2.16, SW2.9
- net INVERTX: now also N_5.19 (Q7)
- net INVERTY: now also N_5.16 (Q6)
- net PL1LED: now also R165.1
- net PL2LED: now also R164.1
- net PR221: now also N_8.11 (LD), P_9.11 (LD), R_10.1 (~1CLR), R_10.10 (~1PRE_), R_10.13 (~1CLR), R_10.4 (~1PRE_)
- net R\~W~B: now also F_5.13
- net ~CONTROL: now also F_5.12
- net ~NVRAM: now also F/H_4.3, N_4.4
- net ~RECALL: now also R171.1, R_3.10 (~RC)
- net at N_9.11 (I0b): now also P_9.7 (QD)
- net at N_9.13 (I1b): now also P_9.6 (QC)
- net at N_9.15 (I2b): now also P_9.3 (QA)
- net at N_9.17 (I3b): now also P_9.2 (QB)
- net at N_9.2 (I0a): now also N_8.7 (QD)
- net at N_9.4 (I1a): now also N_8.6 (QC)
- net at N_9.6 (I2a): now also N_8.3 (QA)
- net at N_9.8 (I3a): now also N_8.2 (QB)
- net at P_9.14 (CK): now also P_10.7 (2Y), R_10.3 (1CLK)
- net at P_9.5 (D/U): now also R_10.5 (1Q)
- net at N_8.14 (CK): now also P_10.12 (4Y), R_10.11 (2CLK)
- net at N_8.5 (D/U): now also R_10.9 (2Q)
- new net: P_10.4 (1Y), R_10.2 (1D)
- new net: P_10.9 (3Y), R_10.12 (2D)
- new net: P_10.10 (3B), P_11.10
- new net: N_10.6, P_10.11 (3A)
- new net: P_10.13 (4B), P_11.8
- new net: N_10.12, P_10.14 (4A)
- new net: N_10.2, P_10.2 (1A)
- new net: P_10.3 (1B), P_11.6
- new net: N_10.4, P_10.5 (2A)
- new net: P_10.6 (2B), P_11.4
- new net: C53.1, N_10.1, R120.1
- new net: N_10.10, R119.1
- new net: C51.1, N_10.11, R118.2, R119.2
- new net: C54.1, P_11.5, R121.2
- new net: C55.1, N_10.3, R122.1
- new net: C56.1, P_11.3, R123.2
- new net: C57.1, N_10.5, R124.1
- new net: C58.1, P_11.11, R125.2
- new net: C59.1, N_10.13, R126.1
- new net: C60.1, P_11.9, R127.2
- new net: C61.1, P_11.1, R128.2, R129.2
- new net: P_11.2, R129.1
- new net: C52.1, R118.1, R120.2, R122.2, R124.2, R126.2
- new net: C62.1, R121.1, R123.1, R125.1, R127.1, R128.1
- new net: N_4.6, R_3.11 (~WE)
- new net: P_4.6, R172.1, R_3.7 (~CS)
- new net: P_4.11, P_4.4, R170.1, R_3.9 (~STR)
- new net: F/H_4.4, P_4.5
- new net: C71.1, N_5.1 (C), R163.2
- new net: F_5.11, N_5.11 (CK)
- new net: M_4.13, N_5.12 (Q4)
- new net: M_4.1, N_5.15 (Q5)
- new net: N_5.2 (Q0), R166.2, R167.2
- new net: N_5.9 (Q3), R168.2, R169.2
- new net: M_4.12, R164.2
- new net: M_4.2, R165.2
- new net: Q15.1 (B), R167.1
- new net: Q16.1 (B), R169.1
- new net: B_2/3.10 (P4), SW1.5
- new net: B_2/3.11 (P5), SW1.6
- new net: B_2/3.12 (P2), SW1.3
- new net: B_2/3.13 (P3), SW1.4
- new net: B_2/3.14 (P0), SW1.1
- new net: B_2/3.15 (P1), SW1.2
- new net: B_2/3.8 (P6), SW1.7
- new net: B_2/3.9 (P7), SW1.8
- new net: D_2/3.10 (P4), SW2.5
- new net: D_2/3.11 (P5), SW2.6
- new net: D_2/3.12 (P2), SW2.3
- new net: D_2/3.13 (P3), SW2.4
- new net: D_2/3.14 (P0), SW2.1
- new net: D_2/3.15 (P1), SW2.2
- new net: D_2/3.8 (P6), SW2.7
- new net: D_2/3.9 (P7), SW2.8
- new net FLIP: N_5.5 (Q1), P_10.1 (S)
- new net POR: P_4.13
- new net R\~WB: N_4.5
- new net UPDATE: N_5.6 (Q2), P_4.12
- no-connect marks 32 -> 38
Other:
- note added: "COIN DOOR AND CONTROL PANEL OUTPUT"
- note added: "NON-VOLATILE MEMORY"
- note added: "TRACK BALL INPUT"
- moved on the sheet: B_1, C64, C65, C67, C68, C69, C70, C74, CR6, D_1, E_1, F/H_4A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

Commit message: Completed 9 pages of schematics
Parts:
- added A_3, C_3: LM324A, symbol Amplifier_Operational:LM324A
- added C78, C79, C81, C91, C92, C93, C94, C95: .1uf, symbol Device:C
- added C80: .022uf, symbol Device:C
- added D_7: LS175C, symbol Star_Wars_Vector_PCB:LS175C
- added E_7: LS157B, symbol Star_Wars_Vector_PCB:LS157B
- added unit 4 of F/H_4
- added F_7: S289, symbol quantum_arcade_pcb:S289
- added K_8: LS32, symbol Star_Wars_Vector_PCB:LS32
- added L2, L3, L4: 1uH, symbol Device:L
- added Q10, Q11, Q9: 2N3904, TO_SOT_Packages_THT:TO-92_Molded_Narrow, symbol Star_Wars_Vector_PCB-rescue:2N3904
- added R130, R132: 1.8k, symbol Device:R_US
- added R131, R133, R135: 2.2k, symbol Device:R_US
- added R134: 3.3k, symbol Device:R_US
- added R136: 6.8k, symbol Device:R_US
- added R137, R138, R139: 470, symbol Device:R_US
- added R188, R189, R190, R191, R192, R193, R194, R195, R196, R197, R198, R199, R200, R201, R202, R203: 4.7k, symbol Device:R_US
- added R204, R206, R207, R208, R209, R211, R212, R213: 220k, symbol Device:R_US
- added R205, R210: 1k, symbol Device:R_US
- added R224, R225, R226: 100, symbol Device:R_US
- added TPAUD1, TPAUD2, TPBLU1, TPGRN1, TPRED1: TP, symbol Star_Wars_Vector_PCB:TP
Connections:
- net +15V: now also A_3.4 (V+), C92.1, C94.1, C_3.4 (V+)
- net +5V: now also D_7.16 (VCC), E_7.16 (VCC), F_7.16 (VCC), R188.1, R189.1, R190.1, R191.1, R192.1, R193.1, R194.1, R195.1, R196.2, R197.2, R198.2, R199.2, R200.2, R201.2, R202.2, R203.2, R204.1
- net -15V: now also A_3.11 (V-), C91.1, C93.1, C_3.11 (V-)
- net AB1: now also B_2/3.36 (A0), D_2/3.36 (A0), E_7.14 (4A)
- net AB2: now also B_2/3.35 (A1), D_2/3.35 (A1), E_7.11 (3A)
- net AB3: now also B_2/3.34 (A2), D_2/3.34 (A2), E_7.5 (2A)
- net AB4: now also B_2/3.33 (A3), D_2/3.33 (A3), E_7.2 (1A)
- net AB5: now also D_2/3.30 (~CSO), F/H_4.9
- net AUDIO+: now also A_3.8, R207.1, R208.2, TPAUD1.1, TPAUD1.2
- net BLUE: now also L3.2, TPBLU1.1, TPBLU1.2
- net CS: now also B_2/3.31 (CS), D_2/3.31 (CS)
- net DB0: now also F_7.~ (I3)
- net DB1: now also F_7.~ (I3)
- net DB2: now also F_7.~ (I3)
- net DB3: now also F_7.~ (I3)
- net DVY0: now also D_7.12 (D2)
- net DVY1: now also D_7.13 (D3)
- net DVY2: now also D_7.5 (D1)
- net DVY3: now also D_7.4 (D0)
- net E: now also B_2/3.7 (PHI2), D_2/3.7 (PHI2)
- net GND: now also A_3.10 (+), A_3.3 (+), C78.1, C91.2, C92.2, C93.2, C94.2, C_3.5 (+), D_7.8 (GND), E_7.15 (E), E_7.8 (GND), F_7.2 (CE), F_7.8 (GND), R137.2, R138.2, R139.2
- net GREEN: now also L4.2, TPGRN1.1, TPGRN1.2
- net RED: now also L2.2, TPRED1.1, TPRED1.2
- net R\~W~B: now also B_2/3.32 (R/~W), D_2/3.32 (R/~W)
- net ~AUDIO: now also A_3.1, R209.1, TPAUD2.1, TPAUD2.2
- net ~COLORAM: now also E_7.1 (S)
- net ~DVY11: now also K_8.13
- net at B_2/3.10 (P4), SW1.5: now also R191.2
- net at B_2/3.11 (P5), SW1.6: now also R190.2
- net at B_2/3.12 (P2), SW1.3: now also R193.2
- net at B_2/3.13 (P3), SW1.4: now also R192.2
- net at B_2/3.14 (P0), SW1.1: now also R195.2
- net at B_2/3.15 (P1), SW1.2: now also R194.2
- net at B_2/3.30 (~CSO): now also F/H_4.8
- net at B_2/3.37 (AUD): now also A_3.6 (-), R205.2
- net at B_2/3.8 (P6), SW1.7: now also R189.2
- net at B_2/3.9 (P7), SW1.8: now also R188.2
- net at D_2/3.10 (P4), SW2.5: now also R199.1
- net at D_2/3.11 (P5), SW2.6: now also R198.1
- net at D_2/3.12 (P2), SW2.3: now also R201.1
- net at D_2/3.13 (P3), SW2.4: now also R200.1
- net at D_2/3.14 (P0), SW2.1: now also R203.1
- net at D_2/3.15 (P1), SW2.2: now also R202.1
- net at D_2/3.37 (AUD): now also C_3.9 (-), R210.2
- net at D_2/3.8 (P6), SW2.7: now also R197.1
- net at D_2/3.9 (P7), SW2.8: now also R196.1
- new net: A_3.7, C79.1, R205.1
- new net: C79.2, R206.2
- new net: C95.1, C_3.8, R210.1
- new net: C95.2, R211.2
- new net: C80.1, C_3.6 (-), R211.1, R212.2
- new net: C80.2, C81.1, C_3.7, R212.1
- new net: C81.2, R213.1
- new net: A_3.9 (-), R206.1, R207.2, R213.2
- new net: A_3.2 (-), R208.1, R209.2
- new net: D_7.10 (Q2), E_7.13 (4B)
- new net: D_7.15 (Q3), E_7.10 (3B)
- new net: D_7.2 (Q0), E_7.3 (1B)
- new net: D_7.7 (Q1), E_7.6 (2B)
- new net: D_7.9 (CK), K_8.11
- new net: E_7.12 (4Y), F_7.~ (I3)
- new net: E_7.4 (1Y), F_7.~ (I3)
- new net: E_7.7 (2Y), F_7.~ (I3)
- new net: E_7.9 (3Y), F_7.~ (I3)
- new net: F_7.11 (D3), R130.2
- new net: F_7.5 (D0), R136.2
- new net: F_7.7 (D1), R134.2
- new net: F_7.9 (D2), R132.2
- new net: Q9.2 (B), R130.1, R131.2
- new net: Q9.1 (E), R137.1, R224.1
- new net: Q10.1 (E), R138.1, R225.1
- new net: Q10.2 (B), R132.1, R133.1
- new net: Q11.1 (E), R139.1, R226.1
- new net: Q11.2 (B), R134.1, R135.1, R136.1
- new net: L4.1, R226.2
- new net: L3.1, R225.2
- new net: L2.1, R224.2
- new net AREF: A_3.5 (+), C78.2, C_3.10 (+), R204.2
- new net ZREF: Q10.3 (C), Q11.3 (C), Q9.3 (C), R131.1, R133.2, R135.2
- new net ~COLORAMWA: F_7.3 (WE)
- new net ~DISRST: D_7.1 (C)
- new net ~STATCLK: K_8.12
- no-connect marks 38 -> 42
Other:
- note added: "AUDIO OUTPUT"
- note added: "COLOR MEMORY AND OUTPUT"
- moved on the sheet: B_2/3, D_2/3, SW1, SW2

Commit message: Completed 10 pages of schematics
Parts:
- added A_7, A_8, B_7, B_8, C_7, C_8: LS194, symbol quantum_arcade_pcb:LS194
- added D/E_4, E/F_4: LS245, symbol Star_Wars_Vector_PCB:LS245
- added D_5, D_6, E_5, E_6: 2KX8_RAM, symbol quantum_arcade_pcb:2KX8_RAM
- added unit 3 of F_5
- added unit 4 of J_10
- added unit 2 of J_10
- added N_6: S02, symbol Star_Wars_Vector_PCB:LS02
- added P_5: LS74, symbol Star_Wars_Vector_PCB:LS74
- added P_6: LS02, symbol Star_Wars_Vector_PCB:LS02
Connections:
- net +5V: now also A_7.16 (VCC), A_8.16 (VCC), B_7.16 (VCC), B_8.16 (VCC), C_7.16 (VCC), C_8.16 (VCC), D/E_4.20 (VCC), D_5.24 (VCC), D_6.24 (VCC), E/F_4.20 (VCC), E_5.24 (VCC), E_6.24 (VCC), P_5.14 (VCC)
- net 1.5M: now also P_6.12
- net 12M: now also A_7.11 (CK), A_8.11 (CK), B_7.11 (CK), B_8.11 (CK), C_7.11 (CK), C_8.11 (CK)
- net 3M: now also P_6.11
- net 6M: now also P_5.11 (2CLK), P_5.3 (1CLK)
- net AS: now also P_5.10 (~1PRE_)
- net DB0: now also B_2/3.38 (D0), D_2/3.38 (D0), D/E_4.11 (B7)
- net DB1: now also B_2/3.39 (D1), D_2/3.39 (D1), D/E_4.12 (B6)
- net DB10: now also E/F_4.13 (B5)
- net DB11: now also E/F_4.14 (B4)
- net DB12: now also E/F_4.15 (B3)
- net DB13: now also E/F_4.16 (B2)
- net DB14: now also E/F_4.17 (B1)
- net DB15: now also E/F_4.18 (B0)
- net DB2: now also B_2/3.40 (D2), D_2/3.40 (D2), D/E_4.13 (B5)
- net DB3: now also B_2/3.2 (D3), D_2/3.2 (D3), D/E_4.14 (B4)
- net DB4: now also B_2/3.3 (D4), D_2/3.3 (D4), D/E_4.15 (B3)
- net DB5: now also B_2/3.4 (D5), D_2/3.4 (D5), D/E_4.16 (B2)
- net DB6: now also B_2/3.5 (D6), D_2/3.5 (D6), D/E_4.17 (B1)
- net DB7: now also B_2/3.6 (D7), D_2/3.6 (D7), D/E_4.18 (B0)
- net DB8: now also E/F_4.11 (B7)
- net DB9: now also E/F_4.12 (B6)
- net DVX10: now also B_8.14 (QB)
- net DVX2: now also A_8.14 (QB)
- net DVX3: now also A_8.15 (QA), C_8.7 (L)
- net DVX4: now also C_8.12 (QD)
- net DVX5: now also C_8.13 (QC)
- net DVX6: now also C_8.14 (QB)
- net DVX7: now also B_8.7 (L), C_8.15 (QA)
- net DVX8: now also B_8.12 (QD)
- net DVX9: now also B_8.13 (QC)
- net DVY0: now also A_7.12 (QD)
- net DVY1: now also A_7.13 (QC)
- net DVY10: now also B_7.14 (QB)
- net DVY2: now also A_7.14 (QB)
- net DVY3: now also A_7.15 (QA)
- net DVY4: now also C_7.12 (QD)
- net DVY5: now also C_7.13 (QC)
- net DVY6: now also C_7.14 (QB)
- net DVY7: now also C_7.15 (QA)
- net DVY8: now also B_7.12 (QD)
- net DVY9: now also B_7.13 (QC)
- net GND: now also A_7.7 (L), A_7.8 (GND), A_8.7 (L), A_8.8 (GND), B_7.8 (GND), B_8.8 (GND), C_7.8 (GND), C_8.8 (GND), D/E_4.10 (GND), D_5.12 (GND), D_5.20 (~OE), D_6.12 (GND), D_6.20 (~OE), E/F_4.10 (GND), E_5.12 (GND), E_5.20 (~OE), E_6.12 (GND), E_6.20 (~OE), P_5.7 (GND)
- net PR219: now also P_5.1 (~1CLR), P_5.13 (~1CLR), P_5.4 (~1PRE_)
- net PR222: now also A_7.1 (C), A_7.2 (R), A_8.2 (R), B_7.1 (C), B_7.2 (R), B_8.2 (R), C_7.1 (C), C_7.2 (R), C_8.2 (R)
- net R\~W: now also D/E_4.1 (DIR), E/F_4.1 (DIR), F_5.9
- net ~DVX11: now also J_10.8
- net ~DVY11: now also J_10.4
- net ~VBUFEN: now also D/E_4.19 (CE), E/F_4.19 (CE), F_5.10, P_5.9 (2Q)
- net ~VMEM: now also N_6.6, P_6.5
- new net: P_5.2 (1D), P_6.13
- new net: P_5.6 (~1Q), P_6.6
- new net: P_6.4, P_6.8
- new net: N_6.4, P_6.9
- new net: D_5.21 (~WE), D_6.21 (~WE), E_5.21 (~WE), E_6.21 (~WE), F_5.8
- new net AM1: D_5.8 (A0), D_6.8 (A0), E_5.8 (A0), E_6.8 (A0)
- new net AM10: D_5.22 (A9), D_6.22 (A9), E_5.22 (A9), E_6.22 (A9)
- new net AM11: D_5.19 (A10), D_6.19 (A10), E_5.19 (A10), E_6.19 (A10)
- new net AM2: D_5.7 (A1), D_6.7 (A1), E_5.7 (A1), E_6.7 (A1)
- new net AM3: D_5.6 (A2), D_6.6 (A2), E_5.6 (A2), E_6.6 (A2)
- new net AM4: D_5.5 (A3), D_6.5 (A3), E_5.5 (A3), E_6.5 (A3)
- new net AM5: D_5.4 (A4), D_6.4 (A4), E_5.4 (A4), E_6.4 (A4)
- new net AM6: D_5.3 (A5), D_6.3 (A5), E_5.3 (A5), E_6.3 (A5)
- new net AM7: D_5.2 (A6), D_6.2 (A6), E_5.2 (A6), E_6.2 (A6)
- new net AM8: D_5.1 (A7), D_6.1 (A7), E_5.1 (A7), E_6.1 (A7)
- new net AM9: D_5.23 (A8), D_6.23 (A8), E_5.23 (A8), E_6.23 (A8)
- new net DVG0: A_7.6 (D), A_8.6 (D), D/E_4.9 (A7), D_5.9 (D0), D_6.9 (D0)
- new net DVG1: A_7.5 (C), A_8.5 (C), D/E_4.8 (A6), D_5.10 (D1), D_6.10 (D1)
- new net DVG10: B_7.4 (B), B_8.4 (B), E/F_4.7 (A5), E_5.11 (D2), E_6.11 (D2)
- new net DVG11: B_7.3 (A), B_8.3 (A), E/F_4.6 (A4), E_5.13 (D3), E_6.13 (D3)
- new net DVG12: E/F_4.5 (A3), E_5.14 (D4), E_6.14 (D4)
- new net DVG13: E/F_4.4 (A2), E_5.15 (D5), E_6.15 (D5)
- new net DVG14: E/F_4.3 (A1), E_5.16 (D6), E_6.16 (D6)
- new net DVG15: E/F_4.2 (A0), E_5.17 (D7), E_6.17 (D7)
- new net DVG2: A_7.4 (B), A_8.4 (B), D/E_4.7 (A5), D_5.11 (D2), D_6.11 (D2)
- new net DVG3: A_7.3 (A), A_8.3 (A), C_7.7 (L), D/E_4.6 (A4), D_5.13 (D3), D_6.13 (D3)
- new net DVG4: C_7.6 (D), C_8.6 (D), D/E_4.5 (A3), D_5.14 (D4), D_6.14 (D4)
- new net DVG5: C_7.5 (C), C_8.5 (C), D/E_4.4 (A2), D_5.15 (D5), D_6.15 (D5)
- new net DVG6: C_7.4 (B), C_8.4 (B), D/E_4.3 (A1), D_5.16 (D6), D_6.16 (D6)
- new net DVG7: B_7.7 (L), C_7.3 (A), C_8.3 (A), D/E_4.2 (A0), D_5.17 (D7), D_6.17 (D7)
- new net DVG8: B_7.6 (D), B_8.6 (D), E/F_4.9 (A7), E_5.9 (D0), E_6.9 (D0)
- new net DVG9: B_7.5 (C), B_8.5 (C), E/F_4.8 (A6), E_5.10 (D1), E_6.10 (D1)
- new net DVX11: B_8.15 (QA), J_10.9
- new net DVY11: B_7.15 (QA), J_10.3
- new net VRAM0: D_5.18 (~CE), E_5.18 (~CE)
- new net VRAM1: D_6.18 (~CE), E_6.18 (~CE)
- new net ~LATCH1: A_8.1 (C), B_8.1 (C), C_8.1 (C)
- new net ~V68K: N_6.5, P_5.12 (2D), P_6.10
- no-connect marks 42 -> 46
Other:
- note added: "BIDIRECTIONAL VECTOR\nMEMORY DATA BUFFERS"
- note added: "VECTOR MEMORY"
- note added: "VECTOR MEMORY ARBITRATOR"
- moved on the sheet: C71, C72, C73, F_5D, M_4A, M_4F, N_5, Q15, Q16, R163, R164, R165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
