File: quantum_arcade_pcb/quantum_arcade_pcb.sch (KiCad schematic (older format))
At the start: 474 parts, among them J20 J20, Q10 2N3904, Q11 2N3904, Q12 2N3906, Q13 2N3904, Q14 2N3904, Q15 2N6044, Q16 2N6044, Q17 2N3904, Q7 2N3904, Q8 2N3906, Q9 2N3904, SW1 SW_DIP_x08, SW2 SW_DIP_x08, Y1 12.096MHz

Commit message: 50 components left to place
Parts:
- removed TPGND4, TPGND5, TPGND6: TP, symbol Star_Wars_Vector_PCB:TP
- added CR4: 1N100, quantum_arcade_pcb:Diode, symbol Device:D
- C19, C31, C49, R54, R81, R82, R83, RV1, RV2: footprint (none) -> quantum_arcade_pcb:GenComp
- C21, C37, C38: footprint (none) -> quantum_arcade_pcb:CapSmall
- C25, C8, R108: footprint (none) -> quantum_arcade_pcb:CapInt
- CR1, CR3, CR5: footprint (none) -> quantum_arcade_pcb:Diode
- Q7, Q8: footprint (none) -> quantum_arcade_pcb:GenTrans
- TP+15V1, TP-15V1, TP5V2, TP6.8V1, TPGND3, TPXOUT1, TPYOUT1: footprint (none) -> quantum_arcade_pcb:TP
Connections:
- net -15V: now also CR4.2 (A)
- net GND: now also CR4.1 (K)
Changed lines of the file:
@@
 F 0 "CR3" V 3554 3004 50  0000 L CNN
 F 1 "1N100" V 3645 3004 50  0000 L CNN
-F 2 "" H 3600 2925 50  0001 C CNN
+F 2 "quantum_arcade_pcb:Diode" H 3600 2925 50  0001 C CNN
 F 3 "~" H 3600 2925 50  0001 C CNN
 	1    3600 2925
@@
 F 0 "TP-15V1" H 3519 1542 60  0000 L CNN
 F 1 "TP" H 3325 1600 60  0001 C CNN
-F 2 "" H 3325 1500 60  0001 C CNN
+F 2 "quantum_arcade_pcb:TP" H 3325 1500 60  0001 C CNN
 F 3 "" H 3325 1500 60  0001 C CNN
 	1    3400 1550
@@
 	3600 3100 3050 3100
 Wire Wire Line
-	3475 1800 3775 1800
+	3475 1800 3675 1800
 Connection ~ 3050 3100
 Wire Wire Line
@@
 F 0 "R108" V 3825 2650 50  0000 C CNN
 F 1 "270" V 3825 2850 50  0000 C CNN
-F 2 "" V 3940 2740 50  0001 C CNN
+F 2 "quantum_arcade_pcb:CapInt" V 3940 2740 50  0001 C CNN
 F 3 "~" H 3900 2750 50  0001 C CNN
 	1    3900 2750
@@
 F 0 "TP+15V1" H 3400 2625 60  0000 L CNN
 F 1 "TP" H 3225 2550 60  0001 C CNN
-F 2 "" H 3225 2450 60  0001 C CNN
+F 2 "quantum_arcade_pcb:TP" H 3225 2450 60  0001 C CNN
 F 3 "" H 3225 2450 60  0001 C CNN
 	1    3300 2500
@@
 F 0 "CR5" V 4204 3004 50  0000 L CNN
 F 1 "1N754A" V 4295 3004 50  0000 L CNN
-F 2 "" H 4250 2925 50  0001 C CNN
+F 2 "quantum_arcade_pcb:Diode" H 4250 2925 50  0001 C CNN
 F 3 "~" H 4250 2925 50  0001 C CNN
 	1    4250 2925
@@
 F 0 "C49" H 4865 2971 50  0000 L CNN
 F 1 ".1uf" H 4865 2880 50  0000 L CNN
-F 2 "" H 4788 2775 50  0001 C CNN
+F 2 "quantum_arcade_pcb:GenComp" H 4788 2775 50  0001 C CNN
 F 3 "~" H 4750 2925 50  0001 C CNN
 	1    4750 2925
@@
 F 0 "TP6.8V1" H 4600 2625 60  0000 L CNN
 F 1 "TP" H 4425 2550 60  0001 C CNN
-F 2 "" H 4425 2450 60  0001 C CNN
+F 2 "quantum_arcade_pcb:TP" H 4425 2450 60  0001 C CNN
 F 3 "" H 4425 2450 60  0001 C CNN
 	1    4500 2500
@@
 F 0 "TP5V2" H 6725 1750 60  0000 L CNN
 F 1 "TP" H 6550 1675 60  0001 C CNN
-F 2 "" H 6550 1575 60  0001 C CNN
+F 2 "quantum_arcade_pcb:TP" H 6550 1575 60  0001 C CNN
 F 3 "" H 6550 1575 60  0001 C CNN
 	1    6625 1625
@@
 F 0 "TPGND3" H 6900 2625 60  0000 L CNN
 F 1 "TP" H 6975 2425 60  0001 C CNN
-F 2 "" H 6975 2325 60  0001 C CNN
+F 2 "quantum_arcade_pcb:TP" H 6975 2325 60  0001 C CNN
 F 3 "" H 6975 2325 60  0001 C CNN
 	1    7050 2375
 	1    0    0    -1
 $EndComp
-$Comp
-L Star_Wars_Vector_PCB:TP TPGND4
-U 1 1 6A60EB5E
-P 7400 2375
-F 0 "TPGND4" H 7250 2625 60  0000 L CNN
-F 1 "TP" H 7325 2425 60  0001 C CNN
-F 2 "" H 7325 2325 60  0001 C CNN
-F 3 "" H 7325 2325 60  0001 C CNN
-	1    7400 2375
-	1    0    0    -1
-$EndComp
-$Comp
-L Star_Wars_Vector_PCB:TP TPGND5
-U 1 1 6A60EEE9
-P 7750 2375
-F 0 "TPGND5" H 7600 2625 60  0000 L CNN
-F 1 "TP" H 7675 2425 60  0001 C CNN
-F 2 "" H 7675 2325 60  0001 C CNN
-F 3 "" H 7675 2325 60  0001 C CNN
-	1    7750 2375
-	1    0    0    -1
-$EndComp
-$Comp
-L Star_Wars_Vector_PCB:TP TPGND6
-U 1 1 6A60F4DC
-P 8100 2375
-F 0 "TPGND6" H 7950 2625 60  0000 L CNN
-F 1 "TP" H 8025 2425 60  0001 C CNN
-F 2 "" H 8025 2325 60  0001 C CNN
-F 3 "" H 8025 2325 60  0001 C CNN
-	1    8100 2375
-	1    0    0    -1
-$EndComp
-Wire Wire Line
-	8175 2575 8175 2625
-Wire Wire Line
-	8175 2625 8025 2625
 Connection ~ 5950 2625
 Wire Wire Line
@@
 Wire Wire Line
 	7125 2575 7125 2625
-Connection ~ 7125 2625
 Wire Wire Line
 	7125 2625 6975 2625
-Wire Wire Line
-	7325 2575 7325 2625
-Connection ~ 7325 2625
-Wire Wire Line
-	7325 2625 7125 2625
-Wire Wire Line
-	7475 2575 7475 2625
-Connection ~ 7475 2625
-Wire Wire Line
-	7475 2625 7325 2625
-Wire Wire Line
-	7675 2575 7675 2625
-Connection ~ 7675 2625
-Wire Wire Line
-	7675 2625 7475 2625
-Wire Wire Line
-	7825 2575 7825 2625
-Connection ~ 7825 2625
-Wire Wire Line
-	7825 2625 7675 2625
-Wire Wire Line
-	8025 2575 8025 2625
-Connection ~ 8025 2625
-Wire Wire Line
-	8025 2625 7825 2625
 $Comp
 L Device:C C96
@@
 F 0 "R54" V 29305 30025 50  0000 C CNN
 F 1 "680" V 29225 30025 50  0000 C CNN
-F 2 "" V 29155 30025 50  0001 C CNN
+F 2 "quantum_arcade_pcb:GenComp" V 29155 30025 50  0001 C CNN
 F 3 "" H 29225 30025 50  0001 C CNN
 	1    29225 30025
@@
 F 0 "C21" H 29050 30475 50  0000 L CNN
 F 1 ".0018uF" H 28900 30275 50  0000 L CNN
-F 2 "" H 29263 30225 50  0001 C CNN
+F 2 "quantum_arcade_pcb:CapSmall" H 29263 30225 50  0001 C CNN
 F 3 "" H 29225 30375 50  0001 C CNN
 	1    29225 30375
@@
 F 0 "C19" H 27950 29175 50  0000 L CNN
 F 1 ".1uF" H 27950 28975 50  0000 L CNN
-F 2 "" H 27963 28925 50  0001 C CNN
+F 2 "quantum_arcade_pcb:GenComp" H 27963 28925 50  0001 C CNN
 F 3 "" H 27925 29075 50  0001 C CNN
 	1    27925 29075
@@
 F 0 "C25" H 30950 29125 50  0000 L CNN
 F 1 ".047uF" H 30950 28925 50  0000 L CNN
-F 2 "" H 30963 28875 50  0001 C CNN
+F 2 "quantum_arcade_pcb:CapInt" H 30963 28875 50  0001 C CNN
 F 3 "" H 30925 29025 50  0001 C CNN
 	1    30925 29025
@@
 F 0 "RV2" V 38725 29000 50  0000 C CNN
 F 1 "VDR" V 38475 29000 50  0000 C CNN
-F 2 "" V 38530 29000 50  0001 C CNN
+F 2 "quantum_arcade_pcb:GenComp" V 38530 29000 50  0001 C CNN
 F 3 "" H 38600 29000 50  0001 C CNN
 	1    38600 29000
@@
 F 0 "TPYOUT1" H 40425 28725 60  0000 C CNN
 F 1 "TP" H 40350 28525 60  0001 C CNN
-F 2 "" H 40350 28425 60  0001 C CNN
+F 2 "quantum_arcade_pcb:TP" H 40350 28425 60  0001 C CNN
 F 3 "" H 40350 28425 60  0001 C CNN
 	1    40425 28475
@@
 F 0 "C31" V 37300 28600 50  0000 L CNN
 F 1 ".1uF" V 37300 28425 50  0000 L CNN
-F 2 "" H 37463 28425 50  0001 C CNN
+F 2 "quantum_arcade_pcb:GenComp" H 37463 28425 50  0001 C CNN
 F 3 "" H 37425 28575 50  0001 C CNN
 	1    37425 28575
@@
 F 0 "C8" H 15975 29150 50  0000 L CNN
 F 1 ".047uF" H 15975 28950 50  0000 L CNN
-F 2 "" H 15988 28900 50  0001 C CNN
+F 2 "quantum_arcade_pcb:CapInt" H 15988 28900 50  0001 C CNN
 F 3 "" H 15950 29050 50  0001 C CNN
 	1    15950 29050
@@
 F 0 "RV1" V 23750 29025 50  0000 C CNN
 F 1 "VDR" V 23500 29025 50  0000 C CNN
-F 2 "" V 23555 29025 50  0001 C CNN
+F 2 "quantum_arcade_pcb:GenComp" V 23555 29025 50  0001 C CNN
 F 3 "" H 23625 29025 50  0001 C CNN
 	1    23625 29025
@@
 F 0 "TPXOUT1" H 25450 28750 60  0000 C CNN
 F 1 "TP" H 25375 28550 60  0001 C CNN
-F 2 "" H 25375 28450 60  0001 C CNN
+F 2 "quantum_arcade_pcb:TP" H 25375 28450 60  0001 C CNN
 F 3 "" H 25375 28450 60  0001 C CNN
 	1    25450 28500
@@
 F 0 "Q7" H 6350 29275 50  0000 L CNN
 F 1 "2N3904" H 6350 29200 50  0000 L CNN
-F 2 "" H 6350 29125 50  0001 L CIN
+F 2 "quantum_arcade_pcb:GenTrans" H 6350 29125 50  0001 L CIN
 F 3 "" H 6150 29200 50  0001 L CNN
 	1    6150 29200
@@
 F 0 "Q8" H 7650 28975 50  0000 L CNN
 F 1 "2N3906" H 7650 28900 50  0000 L CNN
-F 2 "" H 7650 28825 50  0001 L CIN
+F 2 "quantum_arcade_pcb:GenTrans" H 7650 28825 50  0001 L CIN
 F 3 "" H 7450 28900 50  0001 L CNN
 	1    7450 28900
@@
 F 0 "C37" V 5675 29125 50  0000 L CNN
 F 1 "150pF" V 5500 28950 50  0000 L CNN
-F 2 "" H 5663 28925 50  0001 C CNN
+F 2 "quantum_arcade_pcb:CapSmall" H 5663 28925 50  0001 C CNN
 F 3 "" H 5625 29075 50  0001 C CNN
 	1    5625 29075
@@
 F 0 "R81" V 5705 29275 50  0000 C CNN
 F 1 "15K" V 5625 29275 50  0000 C CNN
-F 2 "" V 5555 29275 50  0001 C CNN
+F 2 "quantum_arcade_pcb:GenComp" V 5555 29275 50  0001 C CNN
 F 3 "" H 5625 29275 50  0001 C CNN
 	1    5625 29275
@@
 F 0 "R82" V 6330 28675 50  0000 C CNN
 F 1 "1K" V 6250 28675 50  0000 C CNN
-F 2 "" V 6180 28675 50  0001 C CNN
+F 2 "quantum_arcade_pcb:GenComp" V 6180 28675 50  0001 C CNN
 F 3 "" H 6250 28675 50  0001 C CNN
 	1    6250 28675
@@
 F 0 "C38" V 6800 28875 50  0000 L CNN
 F 1 "39pF" V 6800 28550 50  0000 L CNN
-F 2 "" H 6888 28650 50  0001 C CNN
+F 2 "quantum_arcade_pcb:CapSmall" H 6888 28650 50  0001 C CNN
 F 3 "" H 6850 28800 50  0001 C CNN
 	1    6850 28800
@@
 F 0 "R83" V 6930 29000 50  0000 C CNN
 F 1 "10K" V 6850 29000 50  0000 C CNN
-F 2 "" V 6780 29000 50  0001 C CNN
+F 2 "quantum_arcade_pcb:GenComp" V 6780 29000 50  0001 C CNN
 F 3 "" H 6850 29000 50  0001 C CNN
 	1    6850 29000
@@
 F 0 "CR1" H 8150 30000 50  0000 C CNN
 F 1 "1N914" H 8150 29800 50  0000 C CNN
-F 2 "" H 8150 29900 50  0001 C CNN
+F 2 "quantum_arcade_pcb:Diode" H 8150 29900 50  0001 C CNN
 F 3 "" H 8150 29900 50  0001 C CNN
 	1    8150 29900
@@
 	0    -1   -1   0
 $EndComp
+$Comp
+L Device:D CR4
+U 1 1 989AC1D7
+P 3675 1950
+F 0 "CR4" V 3575 1725 50  0000 L CNN
+F 1 "1N100" V 3700 1625 50  0000 L CNN
+F 2 "quantum_arcade_pcb:Diode" H 3675 1950 50  0001 C CNN
+F 3 "~" H 3675 1950 50  0001 C CNN
+	1    3675 1950
+	0    -1   -1   0
+$EndComp
+Connection ~ 3675 1800
+Wire Wire Line
+	3675 1800 3775 1800
 $EndSCHEMATC
