File: quantum_arcade_pcb/quantum_arcade_pcb.kicad_pcb (KiCad board)
At the start: 2 copper layers, 292.1 x 530.9 mm, 142 parts, among them J20 J20, SW1 SW_DIP_x08, SW2 SW_DIP_x08

Commit message: Placed several components
Parts:
- added C100: .1uf, quantum_arcade_pcb:GenComp, F.Cu at (298.4, 540.4)
- added C101: .1uf, quantum_arcade_pcb:GenComp, F.Cu at (40.0, 485.8)
- added C102: .1uf, quantum_arcade_pcb:GenComp, F.Cu at (64.8, 492.1)
- added C103: .1uf, quantum_arcade_pcb:GenComp, F.Cu at (231.1, 509.3)
- added C104: .1uf, quantum_arcade_pcb:GenComp, F.Cu at (40.0, 442.0)
- added C105: .1uf, quantum_arcade_pcb:GenComp, F.Cu at (64.8, 450.2)
- added C106: .1uf, quantum_arcade_pcb:GenComp, F.Cu at (231.1, 456.6)
- added C129: .1uf, quantum_arcade_pcb:GenComp, F.Cu at (40.0, 159.4)
- added C130: .047uf, quantum_arcade_pcb:GenComp, F.Cu at (300.4, 479.4)
- added C63: 220pf, quantum_arcade_pcb:GenComp, F.Cu at (111.8, 123.2)
- added C64: .1uf, quantum_arcade_pcb:GenComp, F.Cu at (95.2, 178.4)
- added C65: .1uf, quantum_arcade_pcb:GenComp, F.Cu at (95.2, 181.0)
- added C67: .1uf, quantum_arcade_pcb:GenComp, F.Cu at (95.2, 173.4)
- added C68: .1uf, quantum_arcade_pcb:GenComp, F.Cu at (95.2, 165.7)
- added C69: .1uf, quantum_arcade_pcb:GenComp, F.Cu at (95.2, 168.3)
- added C70: .1uf, quantum_arcade_pcb:GenComp, F.Cu at (95.2, 170.8)
- added C78: .1uf, quantum_arcade_pcb:GenComp, F.Cu at (301.0, 508.6)
- added C79: .1uf, quantum_arcade_pcb:GenComp, F.Cu at (300.4, 471.2)
- added C80: .022uf, quantum_arcade_pcb:GenComp, F.Cu at (262.9, 488.9)
- added C81: .1uf, quantum_arcade_pcb:GenComp, F.Cu at (263.5, 494.0)
- added C91: .1uf, quantum_arcade_pcb:GenComp, F.Cu at (300.4, 442.6)
- added C92: .1uf, quantum_arcade_pcb:GenComp, F.Cu at (299.7, 440.1)
- added C93: .1uf, quantum_arcade_pcb:GenComp, F.Cu at (263.5, 445.8)
- added C94: .1uf, quantum_arcade_pcb:GenComp, F.Cu at (262.9, 443.2)
- added C95: .1uf, quantum_arcade_pcb:GenComp, F.Cu at (262.9, 475.0)
- added C96: .1uf, quantum_arcade_pcb:GenComp, F.Cu at (39.4, 540.4)
- added C98: .1uf, quantum_arcade_pcb:GenComp, F.Cu at (189.2, 540.4)
- added C99: .1uf, quantum_arcade_pcb:GenComp, F.Cu at (232.4, 543.6)
- added L1: 100uH, quantum_arcade_pcb:Ind, F.Cu at (44.5, 248.9)
- added L2: 1uH, quantum_arcade_pcb:Ind, F.Cu at (111.1, 70.5)
- added L3: 1uH, quantum_arcade_pcb:Ind, F.Cu at (111.1, 82.5)
- added L4: 1uH, quantum_arcade_pcb:Ind, F.Cu at (111.1, 94.6)
- added Q10: 2N3904, quantum_arcade_pcb:GenTrans, F.Cu at (123.8, 87.0)
- added Q11: 2N3904, quantum_arcade_pcb:GenTrans, F.Cu at (123.8, 97.8)
- added Q12: 2N3906, quantum_arcade_pcb:GenTrans, F.Cu at (123.8, 113.0)
- added Q13: 2N3904, quantum_arcade_pcb:GenTrans, F.Cu at (123.8, 105.4)
- added Q14: 2N3904, quantum_arcade_pcb:GenTrans, F.Cu at (123.8, 123.2)
- added Q9: 2N3904, quantum_arcade_pcb:GenTrans, F.Cu at (123.8, 75.6)
- added R118: 10k, quantum_arcade_pcb:GenComp, F.Cu at (72.4, 137.8)
- added R119: 1k, quantum_arcade_pcb:GenComp, F.Cu at (73.0, 135.3)
- added R120: 10k, quantum_arcade_pcb:GenComp, F.Cu at (72.4, 148.0)
- added R121: 10k, quantum_arcade_pcb:GenComp, F.Cu at (40.0, 144.8)
- added R122: 10k, quantum_arcade_pcb:GenComp, F.Cu at (72.4, 145.4)
- added R123: 10k, quantum_arcade_pcb:GenComp, F.Cu at (40.0, 139.7)
- added R124: 10k, quantum_arcade_pcb:GenComp, F.Cu at (72.4, 142.9)
- added R125: 10k, quantum_arcade_pcb:GenComp, F.Cu at (40.0, 142.2)
- added R126: 10k, quantum_arcade_pcb:GenComp, F.Cu at (73.0, 140.3)
- added R127: 10k, quantum_arcade_pcb:GenComp, F.Cu at (40.0, 147.3)
- added R128: 10k, quantum_arcade_pcb:GenComp, F.Cu at (40.0, 134.6)
- added R129: 1k, quantum_arcade_pcb:GenComp, F.Cu at (40.6, 137.2)
- added R130: 1.8k, quantum_arcade_pcb:GenComp, F.Cu at (111.8, 78.7)
- added R131: 2.2k, quantum_arcade_pcb:GenComp, F.Cu at (111.1, 76.2)
- added R132: 1.8k, quantum_arcade_pcb:GenComp, F.Cu at (111.8, 91.4)
- added R133: 2.2k, quantum_arcade_pcb:GenComp, F.Cu at (111.8, 88.9)
- added R134: 3.3k, quantum_arcade_pcb:GenComp, F.Cu at (111.8, 102.9)
- added R135: 2.2k, quantum_arcade_pcb:GenComp, F.Cu at (111.8, 100.3)
- added R136: 6.8k, quantum_arcade_pcb:GenComp, F.Cu at (111.8, 105.4)
- added R137: 470, quantum_arcade_pcb:GenComp, F.Cu at (111.8, 73.7)
- added R138: 470, quantum_arcade_pcb:GenComp, F.Cu at (111.8, 86.4)
- added R139: 470, quantum_arcade_pcb:GenComp, F.Cu at (111.8, 97.8)
- added R140: 1.2k, quantum_arcade_pcb:GenComp, F.Cu at (94.6, 148.0)
- added R141: 2.2k, quantum_arcade_pcb:GenComp, F.Cu at (94.6, 145.4)
- added R142: 4.7k, quantum_arcade_pcb:GenComp, F.Cu at (111.8, 120.7)
- added R143: 10k, quantum_arcade_pcb:GenComp, F.Cu at (111.8, 118.1)
- added R144: 22k, quantum_arcade_pcb:GenComp, F.Cu at (111.1, 115.6)
- added R145: 3.3k, quantum_arcade_pcb:GenComp, F.Cu at (111.8, 113.0)
- added R146: 510, quantum_arcade_pcb:GenComp, F.Cu at (111.8, 110.5)
- added R147: 1k, quantum_arcade_pcb:GenComp, F.Cu at (111.1, 108.0)
- added R148: 1k, quantum_arcade_pcb:GenComp, F.Cu at (111.8, 125.7)
- added R149: 470, quantum_arcade_pcb:GenComp, F.Cu at (94.6, 137.8)
- added R151: 470, quantum_arcade_pcb:GenComp, F.Cu at (94.6, 142.9)
- added R152: 470, quantum_arcade_pcb:GenComp, F.Cu at (94.6, 140.3)
- added R153: 1k, quantum_arcade_pcb:GenComp, F.Cu at (95.2, 155.6)
- added R155: 1k, quantum_arcade_pcb:GenComp, F.Cu at (95.2, 150.5)
- added R156: 1k, quantum_arcade_pcb:GenComp, F.Cu at (95.2, 153.0)
- added R157: 1k, quantum_arcade_pcb:GenComp, F.Cu at (94.6, 163.2)
- added R158: 1k, quantum_arcade_pcb:GenComp, F.Cu at (95.2, 160.7)
- added R159: 1k, quantum_arcade_pcb:GenComp, F.Cu at (95.2, 158.1)
- added R160: 470, quantum_arcade_pcb:GenComp, F.Cu at (94.6, 130.2)
- added R161: 470, quantum_arcade_pcb:GenComp, F.Cu at (94.6, 132.7)
- added R162: 470, quantum_arcade_pcb:GenComp, F.Cu at (94.6, 135.3)
- added R171: 1k, quantum_arcade_pcb:GenComp, F.Cu at (41.9, 540.4)
- added R172: 1k, quantum_arcade_pcb:GenComp, F.Cu at (40.6, 439.4)
- added R188: 4.7k, quantum_arcade_pcb:GenComp, F.Cu at (300.4, 422.3)
- added R189: 4.7k, quantum_arcade_pcb:GenComp, F.Cu at (300.4, 419.7)
- added R190: 4.7k, quantum_arcade_pcb:GenComp, F.Cu at (300.4, 417.2)
- added R191: 4.7k, quantum_arcade_pcb:GenComp, F.Cu at (300.4, 414.7)
- added R192: 4.7k, quantum_arcade_pcb:GenComp, F.Cu at (300.4, 412.1)
- added R193: 4.7k, quantum_arcade_pcb:GenComp, F.Cu at (300.4, 409.6)
- added R194: 4.7k, quantum_arcade_pcb:GenComp, F.Cu at (300.4, 407.0)
- added R195: 4.7k, quantum_arcade_pcb:GenComp, F.Cu at (300.4, 404.5)
- added R196: 4.7k, quantum_arcade_pcb:GenComp, F.Cu at (268.0, 422.3)
- added R197: 4.7k, quantum_arcade_pcb:GenComp, F.Cu at (268.0, 419.7)
- added R198: 4.7k, quantum_arcade_pcb:GenComp, F.Cu at (268.0, 417.2)
- added R199: 4.7k, quantum_arcade_pcb:GenComp, F.Cu at (268.0, 414.7)
- added R200: 4.7k, quantum_arcade_pcb:GenComp, F.Cu at (268.0, 412.1)
- added R201: 4.7k, quantum_arcade_pcb:GenComp, F.Cu at (268.0, 409.6)
- added R202: 4.7k, quantum_arcade_pcb:GenComp, F.Cu at (268.0, 407.0)
- added R203: 4.7k, quantum_arcade_pcb:GenComp, F.Cu at (268.0, 404.5)
- added R204: 220k, quantum_arcade_pcb:GenComp, F.Cu at (301.0, 511.2)
- added R205: 1k, quantum_arcade_pcb:GenComp, F.Cu at (301.0, 476.9)
- added R206: 220k, quantum_arcade_pcb:GenComp, F.Cu at (300.4, 499.1)
- added R207: 220k, quantum_arcade_pcb:GenComp, F.Cu at (300.4, 484.5)
- added R208: 220k, quantum_arcade_pcb:GenComp, F.Cu at (300.4, 489.6)
- added R209: 220k, quantum_arcade_pcb:GenComp, F.Cu at (300.4, 494.7)
- added R210: 1k, quantum_arcade_pcb:GenComp, F.Cu at (263.5, 471.2)
- added R211: 220k, quantum_arcade_pcb:GenComp, F.Cu at (262.9, 484.5)
- added R212: 220k, quantum_arcade_pcb:GenComp, F.Cu at (262.9, 480.1)
- added R213: 220k, quantum_arcade_pcb:GenComp, F.Cu at (262.9, 498.5)
- added R216: 4.6k, quantum_arcade_pcb:GenComp, F.Cu at (101.0, 440.1)
- added R217: 4.7k, quantum_arcade_pcb:GenComp, F.Cu at (142.9, 438.1)
- added R218: 1k, quantum_arcade_pcb:GenComp, F.Cu at (40.0, 483.2)
- added R221: 1k, quantum_arcade_pcb:GenComp, F.Cu at (47.0, 169.5)
- added TPAUD1: TP, quantum_arcade_pcb:TP, F.Cu at (303.5, 445.1)
- added TPAUD2: TP, quantum_arcade_pcb:TP, F.Cu at (302.3, 437.5)
- added TPGND1: TP, quantum_arcade_pcb:TP, F.Cu at (34.3, 542.3)
- moved N_10 1.27 mm to (77.5, 172.7)
- moved N_8 1.27 mm to (77.5, 248.9)
- moved N_9 1.27 mm to (77.5, 208.9)
- moved N_7 0.63 mm to (78.1, 287.7)
Routing:
- net Net-(L4-Pad1): track 0.00 -> 25.4 mm
- net ZREF: track 0.00 -> 24.1 mm
- net Net-(L2-Pad1): track 0.00 -> 23.5 mm
- net Net-(A_3-Pad7): track 0.00 -> 17.8 mm
- net Net-(B_2/3-Pad14): track 0.00 -> 17.1 mm
- net Net-(B_2/3-Pad13): track 0.00 -> 17.1 mm
- net Net-(B_2/3-Pad11): track 0.00 -> 17.1 mm
- net Net-(L3-Pad1): track 0.00 -> 17.1 mm
- net Net-(B_2/3-Pad8): track 0.00 -> 17.1 mm
- net Net-(B_2/3-Pad15): track 0.00 -> 17.1 mm
- net Net-(B_2/3-Pad9): track 0.00 -> 17.1 mm
- net Net-(B_2/3-Pad12): track 0.00 -> 17.1 mm
- net Net-(B_2/3-Pad10): track 0.00 -> 17.1 mm
- net Net-(Q12-Pad1): track 0.00 -> 14.0 mm
- net Net-(Q12-Pad2): track 0.00 -> 11.4 mm
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Other:
- board text added: "AUD1"
- board text added: "AUD2"
- board text added: "GND"

Commit message: 133 components left to place
Parts:
- added C107: .1uf, quantum_arcade_pcb:GenComp, F.Cu at (39.4, 398.8)
- added C108: .1uf, quantum_arcade_pcb:GenComp, F.Cu at (148.6, 410.8)
- added C109: .1uf, quantum_arcade_pcb:GenComp, F.Cu at (200.0, 406.4)
- added C110: .1uf, quantum_arcade_pcb:GenComp, F.Cu at (300.4, 398.8)
- added C111: .1uf, quantum_arcade_pcb:GenComp, F.Cu at (40.6, 356.2)
- added C112: .1uf, quantum_arcade_pcb:GenComp, F.Cu at (148.6, 367.0)
- added C113: .1uf, quantum_arcade_pcb:GenComp, F.Cu at (189.9, 368.3)
- added C114: .1uf, quantum_arcade_pcb:GenComp, F.Cu at (300.4, 354.3)
- added C115: .1uf, quantum_arcade_pcb:GenComp, F.Cu at (40.0, 311.1)
- added C116: .1uf, quantum_arcade_pcb:GenComp, F.Cu at (109.2, 324.5)
- added C117: .1uf, quantum_arcade_pcb:GenComp, F.Cu at (190.5, 325.1)
- added C118: .1uf, quantum_arcade_pcb:GenComp, F.Cu at (299.7, 312.4)
- added C119: .1uf, quantum_arcade_pcb:GenComp, F.Cu at (40.0, 277.5)
- added C120: .1uf, quantum_arcade_pcb:GenComp, F.Cu at (109.9, 285.8)
- added C121: .1uf, quantum_arcade_pcb:GenComp, F.Cu at (191.1, 285.8)
- added C122: .1uf, quantum_arcade_pcb:GenComp, F.Cu at (301.0, 273.1)
- added C123: .1uf, quantum_arcade_pcb:GenComp, F.Cu at (67.3, 247.0)
- added C124: .1uf, quantum_arcade_pcb:GenComp, F.Cu at (110.5, 247.0)
- added C125: .1uf, quantum_arcade_pcb:GenComp, F.Cu at (191.1, 245.7)
- added C126: .1uf, quantum_arcade_pcb:GenComp, F.Cu at (301.0, 234.9)
- added C127: .1uf, quantum_arcade_pcb:GenComp, F.Cu at (40.6, 196.2)
- added C128: .1uf, quantum_arcade_pcb:GenComp, F.Cu at (151.8, 208.3)
- added C44: 100uf 35V, quantum_arcade_pcb:Cap2, F.Cu at (-3.68, 48.4)
- added C45: 22uf 25V, quantum_arcade_pcb:Cap1, F.Cu at (175.9, 85.1)
- added C46: 100uf 35V, quantum_arcade_pcb:Cap2, F.Cu at (-3.17, 43.8)
- added C47: 22uf 35V, quantum_arcade_pcb:Cap3, F.Cu at (-4.95, 52.7)
- added C48: 22uf 25V, quantum_arcade_pcb:Cap1, F.Cu at (175.9, 129.5)
- added C51: 1000pf 100V, quantum_arcade_pcb:GenComp, F.Cu at (62.2, 95.2)
- added C52: 1uf 50V, quantum_arcade_pcb:Cap1, F.Cu at (67.9, 118.7)
- added C53: 1uf 50V, quantum_arcade_pcb:Cap1, F.Cu at (55.2, 118.7)
- added C54: 1uf 50V, quantum_arcade_pcb:Cap1, F.Cu at (35.6, 95.9)
- added C55: 1uf 50V, quantum_arcade_pcb:Cap1, F.Cu at (55.2, 95.9)
- added C56: 1uf 50V, quantum_arcade_pcb:Cap1, F.Cu at (48.3, 95.9)
- added C57: 1uf 50V, quantum_arcade_pcb:Cap1, F.Cu at (61.6, 118.7)
- added C58: 1uf 50V, quantum_arcade_pcb:Cap1, F.Cu at (41.9, 118.7)
- added C59: 1uf 50V, quantum_arcade_pcb:Cap1, F.Cu at (67.9, 95.9)
- added C60: 1uf 50V, quantum_arcade_pcb:Cap1, F.Cu at (48.3, 118.7)
- added C61: 1000pf 100V, quantum_arcade_pcb:GenComp, F.Cu at (41.9, 95.2)
- added C62: 1uf 50V, quantum_arcade_pcb:Cap1, F.Cu at (35.6, 118.7)
- added C71: .1uf, quantum_arcade_pcb:GenComp, F.Cu at (69.2, 360.7)
- added C72: .1uf, quantum_arcade_pcb:GenComp, F.Cu at (117.5, 160.7)
- added C73: .1uf, quantum_arcade_pcb:GenComp, F.Cu at (117.5, 163.2)
- added C74: 1uf, quantum_arcade_pcb:Cap1, F.Cu at (97.2, 80.0)
- added C75: .1uf, quantum_arcade_pcb:GenComp, F.Cu at (40.6, 221.6)
- added C76: 100pf 100V, quantum_arcade_pcb:CapSmall, F.Cu at (40.6, 249.6)
- added C77: 39pf 100V, quantum_arcade_pcb:CapSmall, F.Cu at (36.8, 249.6)
- added C82: 100uf 25V, quantum_arcade_pcb:Cap2, F.Cu at (94.6, 109.2)
- added C97: .1uf, quantum_arcade_pcb:GenComp, F.Cu at (151.1, 171.4)
- added CR6: 1N100, quantum_arcade_pcb:Diode, F.Cu at (83.2, 92.7)
- added CR7: LED, quantum_arcade_pcb:LED, F.Cu at (80.0, 113.7)
- added Q15: 2N6044, quantum_arcade_pcb:BigTrans, F.Cu at (144.8, 147.3)
- added Q16: 2N6044, quantum_arcade_pcb:BigTrans, F.Cu at (118.1, 146.1)
- added Q17: 2N3904, quantum_arcade_pcb:GenTrans, F.Cu at (36.8, 229.9)
- added R163: 10k, quantum_arcade_pcb:GenComp, F.Cu at (59.7, 355.0)
- added R164: 220, quantum_arcade_pcb:GenComp, F.Cu at (117.5, 175.9)
- added R165: 220, quantum_arcade_pcb:GenComp, F.Cu at (117.5, 178.4)
- added R166: 1k, quantum_arcade_pcb:GenComp, F.Cu at (117.5, 173.4)
- added R167: 1k, quantum_arcade_pcb:GenComp, F.Cu at (117.5, 170.8)
- added R168: 1k, quantum_arcade_pcb:GenComp, F.Cu at (116.8, 168.3)
- added R169: 1k, quantum_arcade_pcb:GenComp, F.Cu at (116.8, 165.7)
- added R170: 1k, quantum_arcade_pcb:GenComp, F.Cu at (48.3, 410.8)
- added R173: 10k, quantum_arcade_pcb:GenComp, F.Cu at (82.5, 82.5)
- added R174: 68k, quantum_arcade_pcb:GenComp, F.Cu at (83.2, 87.6)
- added R175: 15k, quantum_arcade_pcb:GenComp, F.Cu at (83.2, 85.1)
- added R176: 1k, quantum_arcade_pcb:GenComp, F.Cu at (82.5, 90.2)
- added R177: 10k, quantum_arcade_pcb:GenComp, F.Cu at (39.4, 262.3)
- added R178: 10k, quantum_arcade_pcb:GenComp, F.Cu at (38.7, 259.7)
- added R179: 220, quantum_arcade_pcb:GenComp, F.Cu at (38.7, 239.4)
- added R180: 100K, quantum_arcade_pcb:GenComp, F.Cu at (222.2, 242.6)
- added R181: 100K, quantum_arcade_pcb:GenComp, F.Cu at (222.2, 247.7)
- added R182: 100K, quantum_arcade_pcb:GenComp, F.Cu at (222.2, 252.7)
- added R183: 100K, quantum_arcade_pcb:GenComp, F.Cu at (222.2, 257.8)
- added R184: 100K, quantum_arcade_pcb:GenComp, F.Cu at (221.6, 245.1)
- added R185: 100K, quantum_arcade_pcb:GenComp, F.Cu at (221.6, 240.0)
- added R186: 100K, quantum_arcade_pcb:GenComp, F.Cu at (221.6, 255.3)
- added R187: 100K, quantum_arcade_pcb:GenComp, F.Cu at (221.6, 250.2)
- added R214: 1k, quantum_arcade_pcb:GenComp, F.Cu at (80.0, 124.5)
- added R215: 10k, quantum_arcade_pcb:GenComp, F.Cu at (139.1, 400.1)
- added R219: 1k, quantum_arcade_pcb:GenComp, F.Cu at (109.2, 366.4)
- added R220: 1k, quantum_arcade_pcb:GenComp, F.Cu at (47.6, 323.9)
- added R222: 1k, quantum_arcade_pcb:GenComp, F.Cu at (293.4, 247.0)
- added R223: 220, quantum_arcade_pcb:GenComp, F.Cu at (83.2, 95.9)
- added R224: 100, quantum_arcade_pcb:GenComp, F.Cu at (-10.8, 66.0)
- added R225: 100, quantum_arcade_pcb:GenComp, F.Cu at (-10.7, 61.0)
- added R226: 100, quantum_arcade_pcb:GenComp, F.Cu at (-10.8, 71.1)
- added TP12M1: TP, quantum_arcade_pcb:TP, F.Cu at (57.1, 273.1)
- added TPBLU1: TP, quantum_arcade_pcb:TP, F.Cu at (3.81, 61.0)
- added TPGRN1: TP, quantum_arcade_pcb:TP, F.Cu at (3.81, 67.3)
- added TPRED1: TP, quantum_arcade_pcb:TP, F.Cu at (3.81, 73.7)
- added TPRESET1: TP, quantum_arcade_pcb:TP, F.Cu at (82.5, 104.8)
- added TPRESET2: TP, quantum_arcade_pcb:TP, F.Cu at (78.1, 104.8)
- added TPWDDIS1: TP, quantum_arcade_pcb:TP, F.Cu at (135.9, 397.5)
- added VR1: L7815_, quantum_arcade_pcb:BigTrans, F.Cu at (153.7, 94.6)
- added VR2: L7915_, quantum_arcade_pcb:BigTrans, F.Cu at (153.7, 128.3)
- added Y1: 12.096MHz, quantum_arcade_pcb:Crystal, F.Cu at (39.4, 208.9)
- moved L1 0.63 mm to (44.5, 248.3), turned to 90 degrees
Routing:
- net Net-(C71-Pad1): track 0.00 -> 8.89 mm
Other:
- board text added: "12MHZ"
- board text added: "RESET"
- board text added: "WDDIS"

Commit message: 80 components left to place
Parts:
- added C11: .1uF, quantum_arcade_pcb:GenComp, F.Cu at (238.1, 130.2)
- added C15: .1uF, quantum_arcade_pcb:GenComp, F.Cu at (278.1, 130.8)
- added C16: .1uF, quantum_arcade_pcb:GenComp, F.Cu at (301.0, 130.2)
- added C28: .1uF, quantum_arcade_pcb:GenComp, F.Cu at (238.1, 90.2)
- added C33: .1uF, quantum_arcade_pcb:GenComp, F.Cu at (278.8, 90.8)
- added C34: .1uF, quantum_arcade_pcb:GenComp, F.Cu at (295.3, 90.2)
- added C42: 10pF, quantum_arcade_pcb:CapSmall, F.Cu at (258.4, 161.9)
- added R34: 2.7k, quantum_arcade_pcb:GenComp, F.Cu at (273.1, 130.2)
- added R35: 680, quantum_arcade_pcb:GenComp, F.Cu at (270.5, 130.8)
- added R36: 2.2k, quantum_arcade_pcb:GenComp, F.Cu at (245.7, 130.2)
- added R37: 3.9k, quantum_arcade_pcb:GenComp, F.Cu at (265.4, 130.2)
- added R38: 470, quantum_arcade_pcb:GenComp, F.Cu at (248.3, 130.2)
- added R40: 10k, quantum_arcade_pcb:GenComp, F.Cu at (268.0, 130.8)
- added R42: 10k, Star_Wars_Vector_PCB:PotBlk, F.Cu at (288.3, 109.2)
- added R43: 10k, Star_Wars_Vector_PCB:PotBlk, F.Cu at (261.0, 109.2)
- added R44: 2.2k, quantum_arcade_pcb:GenComp, F.Cu at (243.2, 129.5)
- added R45: 2.2k, quantum_arcade_pcb:GenComp, F.Cu at (240.7, 129.5)
- added R47: 2K, Star_Wars_Vector_PCB:PotBlk, F.Cu at (229.2, 109.2)
- added R50: 2.2k, quantum_arcade_pcb:GenComp, F.Cu at (295.9, 130.2)
- added R51: 470, quantum_arcade_pcb:GenComp, F.Cu at (293.4, 130.8)
- added R52: 3.9k, quantum_arcade_pcb:GenComp, F.Cu at (298.4, 130.8)
- added R53: 1k, quantum_arcade_pcb:GenComp, F.Cu at (275.6, 130.8)
- added R60: 2.7k, quantum_arcade_pcb:GenComp, F.Cu at (276.2, 90.8)
- added R61: 680, quantum_arcade_pcb:GenComp, F.Cu at (271.1, 90.8)
- added R63: 470, quantum_arcade_pcb:GenComp, F.Cu at (248.3, 89.5)
- added R64: 2.2k, quantum_arcade_pcb:GenComp, F.Cu at (245.7, 90.2)
- added R65: 3.9k, quantum_arcade_pcb:GenComp, F.Cu at (266.1, 90.2)
- added R67: 10k, quantum_arcade_pcb:GenComp, F.Cu at (268.6, 90.8)
- added R68: 10k, Star_Wars_Vector_PCB:PotBlk, F.Cu at (277.5, 69.8)
- added R69: 2.2k, quantum_arcade_pcb:GenComp, F.Cu at (243.2, 89.5)
- added R70: 2.2k, quantum_arcade_pcb:GenComp, F.Cu at (240.7, 89.5)
- added R72: 10k, Star_Wars_Vector_PCB:PotBlk, F.Cu at (260.4, 69.8)
- added R74: 2K, Star_Wars_Vector_PCB:PotBlk, F.Cu at (229.2, 69.8)
- added R77: 2.2k, quantum_arcade_pcb:GenComp, F.Cu at (297.8, 90.2)
- added R78: 3.9k, quantum_arcade_pcb:GenComp, F.Cu at (302.9, 90.8)
- added R79: 3.9k, quantum_arcade_pcb:GenComp, F.Cu at (300.4, 90.8)
- added R80: 1k, quantum_arcade_pcb:GenComp, F.Cu at (273.7, 90.2)
- added R87: 7.5k, quantum_arcade_pcb:GenComp, F.Cu at (247.0, 163.2)
- added R88: 200, Star_Wars_Vector_PCB:PotBlk, F.Cu at (246.4, 176.5)
- added R89: 7.5K, quantum_arcade_pcb:GenComp, F.Cu at (249.6, 163.2)
- added R91: 7.5k, quantum_arcade_pcb:GenComp, F.Cu at (254.6, 163.2)
- added R92: 200, Star_Wars_Vector_PCB:PotBlk, F.Cu at (262.3, 176.5)
- added R93: 7.5K, quantum_arcade_pcb:GenComp, F.Cu at (252.1, 163.2)
- added TP5V1: TP, quantum_arcade_pcb:TP, F.Cu at (43.8, 52.1)
- added TPGND2: TP, quantum_arcade_pcb:TP, F.Cu at (55.2, 52.1)
- moved C47 165.2 mm to (150.5, 108.6)
- moved C46 154.8 mm to (148.0, 77.5)
- moved C44 153.1 mm to (148.0, 69.8)
- moved R226 145.2 mm to (130.2, 106.0), turned to 90 degrees
- moved R225 144.1 mm to (130.2, 91.4), turned to 90 degrees
- moved R224 141.4 mm to (130.2, 76.8), turned to 90 degrees
- moved TPGRN1 123.4 mm to (124.5, 93.3)
- moved TPBLU1 122.3 mm to (124.5, 81.3)
- moved TPRED1 120.1 mm to (123.8, 70.5)
Other:
- board text added: "+5V"
- board text added: "BLU"
- board text added: "GRN"
- board text added: "RED"
- board text added: "ROM 101/201"
- board text added: "ROM 102"
- board text added: "ROM 103/203"
- board text added: "ROM 104"
- board text added: "ROM 105"
- board text added: "ROM 106/206"
- board text added: "ROM 107"
- board text added: "ROM 108/208"
- board text added: "ROM 109"
- board text added: "ROM 110"

Commit message: 50 components left to place
Parts:
- added C19: .1uF, quantum_arcade_pcb:GenComp, F.Cu at (193.7, 184.8)
- added C21: .0018uF, quantum_arcade_pcb:CapSmall, F.Cu at (189.9, 179.1)
- added C25: .047uF, quantum_arcade_pcb:CapInt, F.Cu at (228.6, 185.4)
- added C31: .1uF, quantum_arcade_pcb:GenComp, F.Cu at (218.4, 88.9)
- added C37: 150pF, quantum_arcade_pcb:CapSmall, F.Cu at (193.7, 123.2)
- added C38: 39pF, quantum_arcade_pcb:CapSmall, F.Cu at (194.3, 134.6)
- added C49: .1uf, quantum_arcade_pcb:GenComp, F.Cu at (218.4, 106.7)
- added C8: .047uF, quantum_arcade_pcb:CapInt, F.Cu at (295.3, 151.1)
- added CR1: 1N914, quantum_arcade_pcb:Diode, F.Cu at (228.0, 203.2)
- added CR3: 1N100, quantum_arcade_pcb:Diode, F.Cu at (191.1, 80.6)
- added CR4: 1N100, quantum_arcade_pcb:Diode, F.Cu at (175.9, 106.7)
- added CR5: 1N754A, quantum_arcade_pcb:Diode, F.Cu at (214.0, 106.7)
- added Q7: 2N3904, quantum_arcade_pcb:GenTrans, F.Cu at (193.0, 111.8)
- added Q8: 2N3906, quantum_arcade_pcb:GenTrans, F.Cu at (193.0, 146.7)
- added R108: 270, quantum_arcade_pcb:CapInt, F.Cu at (214.0, 87.0)
- added R54: 680, quantum_arcade_pcb:GenComp, F.Cu at (193.7, 182.2)
- added R81: 15K, quantum_arcade_pcb:GenComp, F.Cu at (194.3, 126.4)
- added R82: 1K, quantum_arcade_pcb:GenComp, F.Cu at (194.3, 131.4)
- added R83: 10K, quantum_arcade_pcb:GenComp, F.Cu at (193.7, 128.9)
- added RV1: VDR, quantum_arcade_pcb:GenComp, F.Cu at (243.8, 109.9)
- added RV2: VDR, quantum_arcade_pcb:GenComp, F.Cu at (242.6, 69.8)
- added TP+15V1: TP, quantum_arcade_pcb:TP, F.Cu at (196.2, 77.5)
- added TP-15V1: TP, quantum_arcade_pcb:TP, F.Cu at (175.9, 161.3)
- added TP5V2: TP, quantum_arcade_pcb:TP, F.Cu at (180.3, 194.3)
- added TP6.8V1: TP, quantum_arcade_pcb:TP, F.Cu at (208.9, 103.5)
- added TPGND3: TP, quantum_arcade_pcb:TP, F.Cu at (185.4, 67.3)
- added TPXOUT1: TP, quantum_arcade_pcb:TP, F.Cu at (215.9, 120.0)
- added TPYOUT1: TP, quantum_arcade_pcb:TP, F.Cu at (214.0, 75.6)
Other:
- board text added: "+15V"
- board text added: "+6.8V"
- board text added: "-15V"
- board text added: "X OUT"
- board text added: "Y OUT"
