File: quantum_arcade_pcb/quantum_arcade_pcb.kicad_pcb (KiCad board)
At the start: 2 copper layers, 292.1 x 530.9 mm, 486 parts, among them J20 J20, Q10 2N3904, Q11 2N3904, Q12 2N3906, Q13 2N3904, Q14 2N3904, Q15 2N6044, Q16 2N6044, Q17 2N3904, Q7 2N3904, Q8 2N3906, Q9 2N3904, SW1 SW_DIP_x08, SW2 SW_DIP_x08, Y1 12.096MHz

Commit message: 1394 disconnected signals remain
Routing:
- net ~RAM0: track 37.5 -> 294.0 mm, vias 1 -> 2
- net ~RAM1: track 99.7 -> 245.7 mm
- net DB10: track 40.0 -> 177.8 mm, vias 2 -> 3
- net DB13: track 61.6 -> 198.1 mm, vias 2 -> 3
- net DB12: track 51.4 -> 184.8 mm, vias 2 -> 3
- net DB11: track 40.0 -> 168.9 mm, vias 2 -> 3
- net AB7: track 208.9 -> 337.8 mm
- net AB1: track 203.8 -> 308.6 mm
- net AB6: track 205.1 -> 308.6 mm
- net AB3: track 211.5 -> 315.0 mm
- net AB4: track 225.4 -> 328.9 mm
- net AB5: track 216.5 -> 320.0 mm
- net AB8: track 231.8 -> 332.7 mm
- net MB0: track 0.00 -> 85.1 mm
- net ~R~\WB: track 151.8 -> 232.4 mm
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
Commit message: added more traces
Parts:
- moved M_9 1.90 mm to (97.8, 208.9)
- moved R39 1.27 mm to (270.5, 118.1)
- moved R46 1.27 mm to (243.2, 118.1)
- moved C29 1.27 mm to (243.2, 73.7)
- moved C30 1.27 mm to (243.2, 65.4)
- moved R157 0.64 mm to (95.2, 163.2), turned to 180 degrees
Routing:
- net GND: track 6159.7 -> 6440.0 mm, vias 15 -> 22
- net +15V: track 37.5 -> 304.8 mm, vias 0 -> 1
- net +6V: track 5.08 -> 224.8 mm, vias 0 -> 2
- net COINCONTL: track 0.00 -> 162.7 mm, vias 0 -> 1
- net +10V: track 0.00 -> 120.5 mm, vias 0 -> 2
- net 2HORIZCLK: track 0.00 -> 110.0 mm
- net YOUT: track 5.08 -> 110.6 mm
- net 2VERTCLK: track 0.00 -> 100.3 mm
- net 2HORIZDIR: track 0.00 -> 97.0 mm, vias 0 -> 1
- net -15V: track 5.08 -> 101.0 mm
- net 2VERTDIR: track 0.00 -> 95.7 mm, vias 0 -> 1
- net 1HORIZDIR: track 0.00 -> 93.8 mm, vias 0 -> 1
- net 1HORIZCLK: track 0.00 -> 83.3 mm
- net Net-(H_8-Pad15): track 0.00 -> 78.7 mm, vias 0 -> 1
- net 1VERTDIR: track 0.00 -> 77.0 mm, vias 0 -> 1
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
Commit message: 1110 unconnected signals remain
Routing:
- net Net-(CR6-Pad2): track 27.3 -> 271.8 mm, vias 0 -> 1
- net CS: track 0.00 -> 211.5 mm, vias 0 -> 1
- net AB4: track 328.9 -> 520.1 mm, vias 1 -> 3
- net AB3: track 315.0 -> 503.6 mm, vias 0 -> 2
- net AB5: track 320.0 -> 493.4 mm, vias 1 -> 3
- net ~ROM3: track 80.0 -> 243.8 mm, vias 1 -> 2
- net AB1: track 308.6 -> 459.1 mm
- net ~ROM2: track 74.3 -> 205.7 mm, vias 1 -> 2
- net AB11: track 284.5 -> 410.2 mm
- net MB7: track 78.7 -> 204.5 mm
- net AB10: track 288.3 -> 414.0 mm
- net MB6: track 78.7 -> 204.5 mm
- net MB5: track 76.2 -> 201.9 mm
- net ~R~\WB: track 232.4 -> 358.1 mm
- net AB9: track 294.6 -> 420.4 mm
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
Commit message: Added more signal traces
Parts:
- moved C113 2.84 mm to (192.4, 367.0)
- moved L_9 1.91 mm to (119.4, 210.2)
- moved TPGRN1 1.27 mm to (124.5, 92.1)
- moved H_8 1.27 mm to (179.7, 248.9)
- moved C47 0.63 mm to (149.9, 108.6), turned to 180 degrees
- moved H_7 0.63 mm to (179.7, 287.0)
- moved L_8 0.63 mm to (120.7, 248.9)
- turned C48 to 90 degrees
Connections:
- VR2 pad 2: -15V -> -24V
- VR2 pad 3: -24V -> -15V
Routing:
- net -15V: track 149.9 -> 395.0 mm
- net GND: track 6446.3 -> 6690.8 mm, vias 22 -> 24
- net ~AUDIO: track 5.08 -> 247.4 mm, vias 0 -> 1
- net +5V: track 5137.5 -> 5326.0 mm
- net PL2LED: track 0.00 -> 163.2 mm
- net COINCONTR: track 7.15 -> 168.4 mm
- net PL1LED: track 7.25 -> 164.5 mm
- net AUDIO+: track 22.2 -> 170.1 mm, vias 0 -> 2
- net +15V: track 357.5 -> 502.9 mm
- net XOUT: track 34.3 -> 174.4 mm, vias 1 -> 2
- net SELFTEST: track 24.1 -> 158.9 mm
- net START1: track 36.8 -> 170.4 mm
- net COINAUX: track 37.7 -> 166.8 mm
- net COINR: track 17.8 -> 146.0 mm
- net COINL: track 18.7 -> 143.5 mm
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
Commit message: Added ground plane, 786 disconnected signals remain
Parts:
- moved C6 0.64 mm to (264.2, 191.8), turned to 180 degrees
- moved D_7 0.63 mm to (243.8, 287.0)
- moved D_8 0.63 mm to (243.8, 248.9)
Connections:
- J_10 pad 1: INVERTY -> Net-(J_10-Pad1)
- J_10 pad 10: (no net) -> Net-(E_10-Pad1)
- J_10 pad 11: (no net) -> INVERTY
- J_10 pad 2: Net-(E_10-Pad1) -> Net-(J_10-Pad2)
Routing:
- net -15V: track 395.0 -> 1126.5 mm, vias 0 -> 5
- net +15V: track 502.9 -> 1094.7 mm, vias 1 -> 6
- net Net-(B_10-Pad1): track 0.00 -> 239.4 mm
- net INVERTX: track 0.00 -> 239.4 mm, vias 1 -> 2
- net Net-(E_10-Pad15): track 0.00 -> 238.1 mm, vias 0 -> 2
- net ~CENTER: track 0.00 -> 224.8 mm, vias 0 -> 4
- net Net-(C42-Pad2): track 0.00 -> 161.9 mm, vias 0 -> 1
- net XBIP: track 0.00 -> 146.1 mm, vias 0 -> 1
- net VCTR: track 0.00 -> 133.4 mm, vias 0 -> 1
- net YBIP: track 17.8 -> 149.2 mm, vias 0 -> 1
- net INVERTY: track 0.00 -> 125.1 mm, vias 0 -> 2
- net Net-(A_10-Pad7): track 0.00 -> 115.6 mm, vias 0 -> 1
- net DVY3: track 0.00 -> 102.9 mm, vias 0 -> 5
- net YREF: track 0.00 -> 91.4 mm
- net GND: track 6690.8 -> 6775.9 mm
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
Commit message: 592 disconnedted signals remain
Parts:
- moved C112 1.27 mm to (149.9, 367.0)
- moved K_5 1.27 mm to (141.0, 368.9)
- moved C77 1.27 mm to (36.2, 249.6)
- moved C124 1.27 mm to (109.2, 247.0)
- moved C125 1.27 mm to (189.9, 245.7)
- moved K_6 1.27 mm to (141.6, 325.8)
- moved L_8 0.64 mm to (120.0, 248.9)
- moved C76 0.63 mm to (40.6, 249.6)
- moved C97 0.63 mm to (150.5, 171.4)
- moved F_7 0.63 mm to (201.3, 287.0)
- moved K_7 0.63 mm to (141.6, 287.0)
- moved M_8 0.63 mm to (99.1, 248.9)
- moved P_7 0.63 mm to (57.8, 287.0)
- moved R215 0.63 mm to (138.4, 400.1)
- moved TPWDDIS1 0.63 mm to (135.3, 397.5)
Connections:
- H_8 pad 12: Net-(H_8-Pad12) -> Net-(F_8-Pad10)
- H_8 pad 13: Net-(H_8-Pad13) -> Net-(F_8-Pad15)
- H_8 pad 3: Net-(F_8-Pad7) -> Z3
- H_8 pad 5: Net-(F_8-Pad10) -> Net-(F_8-Pad7)
- H_8 pad 6: Net-(F_8-Pad15) -> Z2
- K_8 pad 10: ~DVY11 -> DVY11
- L_6 pad 4: Net-(L_6-Pad4) -> POR
- L_6 pad 5: Net-(L_6-Pad4) -> POR
- L_7 pad 10: CNTR -> VCTR
- L_7 pad 11: VCTR -> CNTR
- P_4 pad 13: ~POR -> POR
- R_4 pad 2: Net-(L_6-Pad4) -> POR
- R_5 pad 2: Net-(L_6-Pad4) -> POR
Routing:
- net PR221: track 16.5 -> 304.8 mm, vias 0 -> 3
- net INVERTX: track 239.4 -> 523.2 mm, vias 2 -> 5
- net ~CENTER: track 224.8 -> 498.5 mm, vias 4 -> 7
- net Net-(N_5-Pad9): track 2.54 -> 273.7 mm, vias 0 -> 4
- net Net-(F_7-Pad11): track 0.00 -> 208.3 mm, vias 0 -> 1
- net DB1: track 120.6 -> 328.9 mm, vias 1 -> 5
- net DB5: track 131.4 -> 334.6 mm, vias 1 -> 2
- net Net-(K_4-Pad13): track 0.00 -> 201.3 mm, vias 0 -> 2
- net Net-(N_5-Pad2): track 0.00 -> 198.1 mm, vias 0 -> 1
- net FLIP: track 0.00 -> 196.8 mm, vias 0 -> 1
- net GND: track 6775.9 -> 6972.3 mm, vias 24 -> 27
- net Net-(J_5-Pad6): track 0.00 -> 196.2 mm, vias 0 -> 1
- net INVERTY: track 125.1 -> 321.3 mm, vias 2 -> 4
- net Net-(F_7-Pad9): track 0.00 -> 195.6 mm, vias 0 -> 1
- net Net-(F_7-Pad7): track 0.00 -> 181.0 mm, vias 0 -> 1
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
Commit message: 542 disconnedted signals remain
Parts:
- moved B_8 0.63 mm to (281.9, 249.6)
- moved C_8 0.63 mm to (264.2, 248.9)
- moved J_7 0.63 mm to (161.3, 287.0)
Connections:
- M_9 pad 12: DB0 -> DB1
- M_9 pad 14: DB1 -> DB0
- N_9 pad 12: DB0 -> DB1
- N_9 pad 14: DB1 -> DB0
Routing:
- net DB0: track 147.3 -> 463.5 mm, vias 0 -> 5
- net ~DISRST: track 37.5 -> 306.5 mm, vias 1 -> 4
- net DVY9: track 74.3 -> 313.7 mm, vias 3 -> 4
- net DVY8: track 67.3 -> 306.1 mm, vias 3 -> 4
- net DB4: track 174.6 -> 412.8 mm, vias 1 -> 3
- net DVY10: track 184.8 -> 398.1 mm, vias 4 -> 5
- net ~LATCH1: track 50.2 -> 241.9 mm, vias 1 -> 2
- net ~TRACKBALL: track 10.2 -> 172.7 mm, vias 0 -> 1
- net DVX10: track 139.7 -> 294.0 mm
- net DVX11: track 97.8 -> 250.8 mm
- net Net-(K_8-Pad2): track 9.53 -> 157.5 mm, vias 1 -> 2
- net DB3: track 236.9 -> 355.6 mm, vias 2 -> 3
- net DB2: track 210.2 -> 321.3 mm, vias 2 -> 3
- net ~VCTR: track 38.1 -> 146.0 mm
- net ~DVX11: track 143.5 -> 246.4 mm
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
Commit message: 495 disconnedted signals remain
Parts:
- moved F_5 1.27 mm to (201.9, 368.9)
- moved F_6 1.27 mm to (201.3, 326.4)
- moved A_7 0.63 mm to (302.3, 287.0)
- moved A_8 0.63 mm to (302.3, 249.6)
- moved B_7 0.63 mm to (281.9, 287.0)
- moved C122 0.63 mm to (300.4, 273.1)
- moved C126 0.63 mm to (300.4, 234.9)
- moved C_7 0.63 mm to (264.2, 287.0)
Routing:
- net DB0: track 463.5 -> 650.2 mm, vias 5 -> 6
- net DVG1: track 0.00 -> 172.7 mm, vias 0 -> 2
- net DVG2: track 0.00 -> 171.5 mm, vias 0 -> 2
- net DVG10: track 0.00 -> 123.8 mm, vias 0 -> 2
- net DVG9: track 0.00 -> 120.7 mm, vias 0 -> 2
- net DVG11: track 15.2 -> 135.3 mm, vias 1 -> 2
- net AB4: track 520.1 -> 634.4 mm, vias 3 -> 6
- net DVG5: track 15.2 -> 125.1 mm
- net DVG6: track 17.8 -> 127.6 mm
- net DVG4: track 14.6 -> 120.0 mm
- net DVG7: track 17.8 -> 123.2 mm
- net DVG13: track 16.5 -> 117.5 mm
- net DVG14: track 17.1 -> 118.1 mm
- net DVG0: track 0.00 -> 100.3 mm, vias 0 -> 1
- net DVG15: track 17.1 -> 116.8 mm
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