File: quantum_arcade_pcb/quantum_arcade_pcb.kicad_pcb (KiCad board)
At the start: 2 copper layers, 292.1 x 530.9 mm, 486 parts, among them J20 J20, Q10 2N3904, Q11 2N3904, Q12 2N3906, Q13 2N3904, Q14 2N3904, Q15 2N6044, Q16 2N6044, Q17 2N3904, Q7 2N3904, Q8 2N3906, Q9 2N3904, SW1 SW_DIP_x08, SW2 SW_DIP_x08, Y1 12.096MHz

Commit message: 388 disconnedted signals remain
Routing:
- net AB2: track 366.4 -> 737.9 mm, vias 0 -> 6
- net DB9: track 56.5 -> 350.5 mm, vias 1 -> 3
- net DB14: track 71.8 -> 358.8 mm, vias 0 -> 2
- net DB4: track 412.8 -> 696.0 mm, vias 3 -> 4
- net DB8: track 61.0 -> 342.3 mm, vias 1 -> 3
- net AB1: track 459.1 -> 732.7 mm, vias 0 -> 6
- net DB15: track 78.1 -> 349.9 mm, vias 0 -> 2
- net DB0: track 650.2 -> 917.6 mm, vias 6 -> 11
- net ~AUDIO: track 246.8 -> 509.0 mm, vias 1 -> 2
- net AUDIO+: track 276.1 -> 534.6 mm, vias 3 -> 4
- net DB1: track 294.6 -> 535.3 mm, vias 3 -> 7
- net AB4: track 634.4 -> 875.0 mm, vias 6 -> 9
- net AB3: track 503.6 -> 741.7 mm, vias 2 -> 6
- net AB5: track 493.4 -> 711.8 mm, vias 3 -> 6
- net GND: track 7042.1 -> 7252.3 mm
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
Commit message: 295 disconnedted signals remain
Parts:
- moved C112 0.64 mm to (149.2, 367.0)
- moved M_7 0.64 mm to (98.4, 287.0)
- moved R219 0.64 mm to (108.6, 366.4)
- moved C117 0.63 mm to (189.9, 325.1)
Connections:
- F_5 pad 13: R\~W~B -> ~WEL
- F_5 pad 2: R\~W~B -> ~WEL
Routing:
- net Net-(L_4-Pad11): track 0.00 -> 278.1 mm, vias 0 -> 2
- net AS: track 318.1 -> 560.1 mm, vias 4 -> 5
- net ~AS: track 342.9 -> 574.7 mm, vias 4 -> 6
- net DB7: track 462.3 -> 682.0 mm
- net Net-(B_1-Pad13): track 170.2 -> 377.8 mm, vias 1 -> 2
- net DB6: track 483.9 -> 689.6 mm, vias 4 -> 5
- net DB5: track 504.8 -> 703.6 mm, vias 3 -> 4
- net SCALE: track 0.00 -> 187.3 mm, vias 0 -> 2
- net ~WEL: track 84.5 -> 270.5 mm, vias 1 -> 3
- net DB2: track 530.2 -> 711.8 mm, vias 6 -> 8
- net ~V68K: track 62.2 -> 237.5 mm, vias 1 -> 4
- net Net-(F_5-Pad11): track 0.00 -> 156.2 mm, vias 0 -> 2
- net ~VBUFEN: track 121.9 -> 273.7 mm, vias 1 -> 3
- net Net-(J_4-Pad1): track 62.9 -> 211.5 mm, vias 1 -> 2
- net Net-(M_4-Pad2): track 113.7 -> 261.0 mm, vias 3 -> 4
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
Commit message: 208 disconnedted signals remain
Parts:
- moved E_7 0.64 mm to (221.0, 287.0)
- moved L_7 0.64 mm to (120.0, 287.0)
- moved C121 0.63 mm to (191.1, 286.4)
Connections:
- B_7 pad 7: DVG7 -> DVY7
- J_5 pad 12: OP0 -> ~OP0
Routing:
- net Net-(A_8-Pad9): track 59.1 -> 287.0 mm, vias 1 -> 2
- net DVY11: track 146.1 -> 346.7 mm
- net 1.5M: track 0.00 -> 200.0 mm, vias 0 -> 1
- net ~AUDIO: track 509.0 -> 707.8 mm
- net AUDIO+: track 534.6 -> 725.7 mm
- net 6M: track 330.8 -> 501.6 mm, vias 4 -> 6
- net Net-(D_7-Pad9): track 30.5 -> 173.4 mm, vias 2 -> 3
- net SCALELO: track 101.6 -> 241.9 mm, vias 3 -> 4
- net 12M: track 238.1 -> 366.4 mm, vias 10 -> 11
- net DVG14: track 162.6 -> 290.2 mm, vias 1 -> 2
- net DVY5: track 152.9 -> 275.4 mm
- net ~COLORAM: track 59.1 -> 179.7 mm, vias 2 -> 4
- net Net-(F_7-Pad7): track 181.0 -> 297.8 mm, vias 1 -> 3
- net DVY4: track 155.6 -> 271.1 mm
- net OP2: track 11.4 -> 125.7 mm, vias 1 -> 3
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
Commit message: 84 disconnected signals remain
Parts:
- moved F_5 0.64 mm to (201.3, 368.9)
Connections:
- C_7 pad 7: DVG3 -> DVY3
- J_7 pad 1: PR222 -> Net-(J_7-Pad1)
- L_8 pad 8: 1.5M -> ST2
Routing:
- net 12M: track 366.4 -> 697.9 mm, vias 11 -> 14
- net Net-(A_7-Pad9): track 10.2 -> 254.6 mm, vias 1 -> 2
- net ST2: track 0.00 -> 218.4 mm, vias 0 -> 4
- net DB3: track 655.3 -> 847.7 mm
- net DB1: track 661.7 -> 850.3 mm
- net DVG8: track 109.9 -> 276.2 mm, vias 1 -> 2
- net ~STROBE0: track 84.5 -> 245.1 mm
- net ~OP0: track 99.1 -> 245.1 mm
- net DB2: track 711.8 -> 854.1 mm
- net Net-(F_6-Pad4): track 40.0 -> 173.4 mm, vias 2 -> 3
- net Net-(A_7-Pad10): track 17.8 -> 144.1 mm
- net OP1: track 54.6 -> 179.1 mm
- net DVG12: track 170.2 -> 285.1 mm, vias 2 -> 4
- net DVG15: track 174.6 -> 278.1 mm, vias 2 -> 4
- net ~VGGO: track 71.8 -> 170.2 mm, vias 1 -> 5
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
Commit message: All signals connected
Connections:
- J_5 pad 10: PR221 -> PR219
Routing:
- net ~VMEM: track 252.1 -> 497.8 mm
- net ~STROBE1: track 154.9 -> 295.3 mm
- net ~V68K: track 370.8 -> 511.2 mm, vias 4 -> 6
- net ~STROBE2: track 75.6 -> 214.0 mm, vias 2 -> 3
- net PR219: track 69.2 -> 204.5 mm
- net ~TRACKBALL: track 228.0 -> 355.6 mm
- net ~OP2: track 137.2 -> 264.2 mm
- net ST3: track 63.5 -> 176.5 mm
- net ST2: track 218.4 -> 318.8 mm
- net VHALT: track 168.9 -> 265.4 mm
- net GND: track 7432.6 -> 7528.5 mm, vias 29 -> 30
- net AM5: track 80.6 -> 174.6 mm, vias 0 -> 2
- net AM6: track 99.1 -> 188.6 mm
- net AM9: track 97.2 -> 184.8 mm
- net AM8: track 78.1 -> 164.5 mm, vias 0 -> 2
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Other:
- board text added: "Designed By Nick Mikstas"
